Commit message: create two loggers prototype

File: loggers_description/urdf/two_loggers.urdf.xacro (robot description, xacro)
@@ -1,8 +1,8 @@
 <?xml version="1.0" ?>
-<robot name="logger" xmlns:xacro="https://www.ros.org/wiki/xacro" >
+<robot name="two_loggers" xmlns:xacro="https://www.ros.org/wiki/xacro" >
   <!-- Constants for robot dimensions -->
   <xacro:property name="PI" value="3.1415926535897931"/>
   <!-- Import all Gazebo-customization elements, including Gazebo colors -->
-  <xacro:include filename="$(find loggers_description)/urdf/single_logger.gazebo" />
+  <xacro:include filename="$(find loggers_description)/urdf/two_loggers.gazebo" />
   <!-- Import Rviz colors -->
   <xacro:include filename="$(find loggers_description)/urdf/materials.xacro" />
@@ -14,31 +14,40 @@
   <!-- </joint> -->
   <link name="link_chassis_1">
-    <collision>
-      <geometry>
-        <box size="0.5 0.3 0.07"/>
-      </geometry>
-    </collision>
-    <visual>
-      <origin rpy="0 0 0" xyz="0 0 0"/>
-      <geometry>
-        <box size="0.5 0.3 0.07"/>
+    <visual>
+      <origin rpy="0 0 0" xyz="0 0 0"/>
+      <geometry>
+        <box size="0.4 0.2 0.1"/>
       </geometry>
       <material name="blue"/>
     </visual>
+    <collision>
+      <origin rpy="0 0 0" xyz="0 0 0"/>
+      <geometry>
+        <box size="0.4 0.2 0.1"/>
+      </geometry>
+    </collision>
     <inertial>
       <mass value="2"/>
       <origin rpy="0 0 0" xyz="0 0 0"/>
-      <inertia ixx="0.01582" ixy="0" ixz="0" iyy="0.04248" iyz="0" izz="0.05667"/>
-    </inertial>
-  </link>
-  <joint name="joint_chassis_caster_1" type="fixed">
+      <inertia ixx="0.0083" ixy="0" ixz="0" iyy="0.0283" iyz="0" izz="0.0333"/>
+    </inertial>
+  </link>
+  <joint name="joint_chassis1_caster1" type="fixed">
     <parent link="link_chassis_1"/>
     <child link="link_caster_1"/>
+    <origin rpy="0 0 0" xyz="0.15 0 -0.05"/>
   </joint>
   <link name="link_caster_1">
-    <collision>
-      <origin rpy=" 0 0 0" xyz="0.2 0 -0.05"/>
-      <geometry>
-        <sphere radius="0.05"/>
+    <visual>
+      <origin rpy="0 0 0" xyz="0 0 0"/>
+      <geometry>
+        <sphere radius="0.04"/>
+      </geometry>
+      <material name="black"/>
+    </visual>
+    <collision>
+      <origin rpy=" 0 0 0" xyz="0 0 0"/>
+      <geometry>
+        <sphere radius="0.04"/>
       </geometry>
       <surface>
@@ -53,26 +62,56 @@
       </surface>
     </collision>
-    <visual>
-      <origin rpy=" 0 0 0" xyz="0.2 0 -0.05"/>
-      <geometry>
-        <sphere radius="0.05"/>
-      </geometry>
-      <material name="black"/>
-    </visual>
-    <inertial>
-      <mass value="0.01"/>
-      <origin rpy="0 0 0" xyz="0 0 0"/>
-      <inertia ixx="0.001" ixy="0" ixz="0" iyy="0.001" iyz="0" izz="0.001"/>
-    </inertial>
-  </link>
-  <joint name="joint_chassis_rwheel_1" type="continuous">
-    <origin rpy="0 0 0" xyz="-0.05 0.15 0"/>
+    <inertial>
+      <mass value="0.02"/>
+      <origin rpy="0 0 0" xyz="0 0 0"/>
+      <inertia ixx="0.00001" ixy="0" ixz="0" iyy="0.00001" iyz="0" izz="0.00001"/>
+    </inertial>
+  </link>
+  <joint name="joint_chassis1_lwheel1" type="continuous">
+    <origin rpy="0 0 0" xyz="-0.16 0.12 0.01"/>
+    <child link="link_left_wheel_1" />
+    <parent link="link_chassis_1"/>
+    <axis rpy="0 0 0" xyz="0 1 0"/>
+  </joint>
+  <link name="link_left_wheel_1">
+    <visual>
+      <origin rpy="${PI/2} 0 0" xyz="0 0 0"/>
+      <geometry>
+        <cylinder length="0.04" radius="0.1"/>
+      </geometry>
+      <material name="orange"/>
+    </visual>
+    <collision>
+      <origin rpy="${PI/2} 0 0" xyz="0 0 0" />
+      <geometry>
+        <cylinder length="0.04" radius="0.1"/>
+      </geometry>
+    </collision>
+    <inertial>
+      <mass value="0.02"/>
+      <origin rpy="0 0 0" xyz="0 0 0"/>
+      <inertia ixx="0.0001" ixy="0" ixz="0" iyy="0.0001" iyz="0" izz="0.0001"/>
+    </inertial>
+  </link>
+  <joint name="joint_chassis1_rwheel1" type="continuous">
+    <origin rpy="0 0 0" xyz="-0.16 -0.12 0.01"/>
     <child link="link_right_wheel_1" />
     <parent link="link_chassis_1"/>
     <axis rpy="0 0 0" xyz="0 1 0"/>
-    <!-- <limit effort="10000" velocity="1000"/> -->
-    <!-- <joint_properties damping="1.0" friction="1.0" /> -->
   </joint>
   <link name="link_right_wheel_1">
+    <collision>
+      <origin rpy="${PI/2} 0 0" xyz="0 0 0" />
+      <geometry>
+        <cylinder length="0.04" radius="0.1"/>
+      </geometry>
+    </collision>
+    <visual>
+      <origin rpy="${PI/2} 0 0" xyz="0 0 0"/>
+      <geometry>
+        <cylinder length="0.04" radius="0.1"/>
+      </geometry>
+      <material name="orange"/>
+    </visual>
     <inertial>
       <mass value="0.01"/>
@@ -80,70 +119,191 @@
       <inertia ixx="0.001" ixy="0" ixz="0" iyy="0.001" iyz="0" izz="0.001"/>
     </inertial>
-    <collision>
-      <origin rpy="0 ${PI/2} ${PI/2}" xyz="0 0 0" />
-      <geometry>
-        <cylinder length="0.04" radius="0.1"/>
-      </geometry>
-    </collision>
-    <visual>
-      <origin rpy="0 ${PI/2} ${PI/2}" xyz="0 0 0"/>
-      <geometry>
-        <cylinder length="0.04" radius="0.1"/>
-      </geometry>
-      <material name="orange"/>
-    </visual>
-  </link>
-  <joint name="joint_chassis_lwheel_1" type="continuous">
-    <origin rpy="0 0 0" xyz="-0.05 -0.15 0"/>
-    <child link="link_left_wheel_1" />
-    <parent link="link_chassis_1"/>
-    <axis rpy="0 0 0" xyz="0 1 0"/>
-    <!-- <limit effort="10000" velocity="1000"/> -->
-    <!-- <joint_properties damping="1.0" friction="1.0" /> -->
-  </joint>
-  <link name="link_left_wheel_1">
-    <collision>
-      <origin rpy="0 ${PI/2} ${PI/2}" xyz="0 0 0" />
-      <geometry>
-        <cylinder length="0.04" radius="0.1"/>
-      </geometry>
-    </collision>
-    <visual>
-      <origin rpy="0 ${PI/2} ${PI/2}" xyz="0 0 0"/>
-      <geometry>
-        <cylinder length="0.04" radius="0.1"/>
-      </geometry>
-      <material name="orange"/>
-    </visual>
-    <inertial>
-      <mass value="0.01"/>
-      <origin rpy="0 0 0" xyz="0 0 0"/>
-      <inertia ixx="0.001" ixy="0" ixz="0" iyy="0.001" iyz="0" izz="0.001"/>
-    </inertial>
-  </link>
-  <joint name="joint_chassis_hat_1" type="continuous">
-    <origin rpy="0 0 0" xyz="0 0 0.04"/>
+  </link>
+  <joint name="joint_chassis1_hat1" type="continuous">
+    <origin rpy="0 0 0" xyz="0.0 0 0.05"/>
     <child link="link_hat_1" />
     <parent link="link_chassis_1"/>
     <axis rpy="0 0 0" xyz="0 0 1"/>
-    <!-- <limit effort="10000" velocity="1000"/> -->
-    <!-- <joint_properties damping="1.0" friction="1.0" /> -->
   </joint>
   <link name="link_hat_1">
-    <collision>
-      <geometry>
-        <cylinder length="0.1" radius="0.02"/>
-      </geometry>
-    </collision>
-    <visual>
-      <origin rpy="0 0 0" xyz="0 0 0"/>
-      <geometry>
-        <cylinder length="0.1" radius="0.02"/>
+    <visual>
+      <origin rpy="0 0 0" xyz="0 0 0.04"/>
+      <geometry>
+        <cylinder length="0.08" radius="0.02"/>
+      </geometry>
+      <material name="orange"/>
+    </visual>
+    <collision>
+      <origin rpy="0 0 0" xyz="0 0 0.04"/>
+      <geometry>
+        <cylinder length="0.08" radius="0.02"/>
+      </geometry>
+    </collision>
+    <inertial>
+      <mass value="0.01"/>
+      <origin rpy="0 0 0" xyz="0 0 0.04"/>
+      <inertia ixx="0.00001" ixy="0" ixz="0" iyy="0.00001" iyz="0" izz="0.00001"/>
+    </inertial>
+  </link>
+  <joint name="joint_hat1_log" type="fixed">
+    <parent link="link_hat_1"/>
+    <child link="link_log"/>
+    <origin rpy="0 0 0" xyz="0 0 0.08"/>
+  </joint>
+  <link name="link_log">
+    <visual>
+      <origin rpy="${PI/2} 0 0" xyz="0 0.8 0"/>
+      <geometry>
+        <cylinder length="1.6" radius="0.01"/>
+      </geometry>
+      <material name="red"/>
+    </visual>
+    <collision>
+      <origin rpy="${PI/2} 0 0" xyz="0 0.8 0"/>
+      <geometry>
+        <cylinder length="1.6" radius="0.01"/>
+      </geometry>
+    </collision>
+    <inertial>
+      <mass value="0.01"/>
+      <origin rpy="${PI/2} 0 0" xyz="0 0.8 0"/>
+      <inertia ixx="0.00001" ixy="0" ixz="0" iyy="0.00001" iyz="0" izz="0.00001"/>
+    </inertial>
+  </link>
+  <joint name="joint_log_hat2" type="fixed">
+    <parent link="link_log"/>
+    <child link="link_hat_2"/>
+    <origin rpy="0 0 0" xyz="0 1.6 0"/>
+  </joint>
+  <link name="link_hat_2">
+    <visual>
+      <origin rpy="0 0 0" xyz="0 0 -0.04"/>
+      <geometry>
+        <cylinder length="0.08" radius="0.02"/>
       </geometry>
       <material name="blue"/>
     </visual>
+    <collision>
+      <origin rpy="0 0 0" xyz="0 0 -0.04"/>
+      <geometry>
+        <cylinder length="0.08" radius="0.02"/>
+      </geometry>
+    </collision>
+    <inertial>
+      <mass value="0.01"/>
+      <origin rpy="0 0 0" xyz="0 0 -0.04"/>
+      <inertia ixx="0.00001" ixy="0" ixz="0" iyy="0.00001" iyz="0" izz="0.00001"/>
+    </inertial>
+  </link>
+  <joint name="joint_chassis2_hat2" type="continuous">
+    <origin rpy="0 0 0" xyz="0.0 0 -0.08"/>
+    <parent link="link_hat_2" />
+    <child link="link_chassis_2"/>
+    <axis rpy="0 0 0" xyz="0 0 1"/>
+  </joint>
+  <link name="link_chassis_2">
+    <visual>
+      <origin rpy="0 0 0" xyz="0 0 -0.05"/>
+      <geometry>
+        <box size="0.4 0.2 0.1"/>
+      </geometry>
+      <material name="orange"/>
+    </visual>
+    <collision>
+      <origin rpy="0 0 0" xyz="0 0 -0.05"/>
+      <geometry>
+        <box size="0.4 0.2 0.1"/>
+      </geometry>
+    </collision>
     <inertial>
       <mass value="2"/>
-      <origin rpy="0 0 0" xyz="0 0 0"/>
+      <origin rpy="0 0 0" xyz="0 0 -0.05"/>
+      <inertia ixx="0.0083" ixy="0" ixz="0" iyy="0.0283" iyz="0" izz="0.0333"/>
+    </inertial>
+  </link>
+  <joint name="joint_chassis2_caster2" type="fixed">
+    <parent link="link_chassis_2"/>
+    <child link="link_caster_2"/>
+    <origin rpy="0 0 0" xyz="0.15 0 -0.1"/>
+  </joint>
+  <link name="link_caster_2">
+    <visual>
+      <origin rpy="0 0 0" xyz="0 0 0"/>
+      <geometry>
+        <sphere radius="0.04"/>
+      </geometry>
+      <material name="white"/>
+    </visual>
+    <collision>
+      <origin rpy=" 0 0 0" xyz="0 0 0"/>
+      <geometry>
+        <sphere radius="0.04"/>
+      </geometry>
+      <surface>
+        <friction>
+          <ode>
+            <mu>0</mu>
+            <mu2>0</mu2>
+            <slip1>1.0</slip1>
+            <slip2>1.0</slip2>
+          </ode>
+        </friction>
+      </surface>
+    </collision>
+    <inertial>
+      <mass value="0.02"/>
+      <origin rpy="0 0 0" xyz="0 0 0"/>
+      <inertia ixx="0.00001" ixy="0" ixz="0" iyy="0.00001" iyz="0" izz="0.00001"/>
+    </inertial>
+  </link>
+  <joint name="joint_chassis2_lwheel2" type="continuous">
+    <origin rpy="0 0 0" xyz="-0.16 0.12 -0.04"/>
+    <child link="link_left_wheel_2" />
+    <parent link="link_chassis_2"/>
+    <axis rpy="0 0 0" xyz="0 1 0"/>
+  </joint>
+  <link name="link_left_wheel_2">
+    <visual>
+      <origin rpy="${PI/2} 0 0" xyz="0 0 0"/>
+      <geometry>
+        <cylinder length="0.04" radius="0.1"/>
+      </geometry>
+      <material name="blue"/>
+    </visual>
+    <collision>
+      <origin rpy="${PI/2} 0 0" xyz="0 0 0" />
+      <geometry>
+        <cylinder length="0.04" radius="0.1"/>
+      </geometry>
+    </collision>
+    <inertial>
+      <mass value="0.02"/>
+      <origin rpy="${PI/2} 0 0" xyz="0 0 0"/>
+      <inertia ixx="0.0001" ixy="0" ixz="0" iyy="0.0001" iyz="0" izz="0.0001"/>
+    </inertial>
+  </link>
+  <joint name="joint_chassis2_rwheel2" type="continuous">
+    <origin rpy="0 0 0" xyz="-0.16 -0.12 -0.04"/>
+    <child link="link_right_wheel_2" />
+    <parent link="link_chassis_2"/>
+    <axis rpy="0 0 0" xyz="0 1 0"/>
+  </joint>
+  <link name="link_right_wheel_2">
+    <collision>
+      <origin rpy="${PI/2} 0 0" xyz="0 0 0" />
+      <geometry>
+        <cylinder length="0.04" radius="0.1"/>
+      </geometry>
+    </collision>
+    <visual>
+      <origin rpy="${PI/2} 0 0" xyz="0 0 0"/>
+      <geometry>
+        <cylinder length="0.04" radius="0.1"/>
+      </geometry>
+      <material name="blue"/>
+    </visual>
+    <inertial>
+      <mass value="0.01"/>
+      <origin rpy="${PI/2} 0 0" xyz="0 0 0"/>
       <inertia ixx="0.001" ixy="0" ixz="0" iyy="0.001" iyz="0" izz="0.001"/>
     </inertial>
