Commit message: recreate two_loggers urdf, started from link_log

File: loggers_description/urdf/two_loggers.urdf.xacro (robot description, xacro)
@@ -1,6 +1,8 @@
 <?xml version="1.0" ?>
+<!-- This model started from link_log -->
 <robot name="two_loggers" xmlns:xacro="https://www.ros.org/wiki/xacro" >
   <!-- Constants for robot dimensions -->
   <xacro:property name="PI" value="3.1415926535897931"/>
+  <xacro:property name="EPSILON" value="1e-6"/> <!-- a small number for default inertia -->
   <!-- Import all Gazebo-customization elements, including Gazebo colors -->
   <xacro:include filename="$(find loggers_description)/urdf/two_loggers.gazebo" />
@@ -9,11 +11,65 @@
   <!-- Use a dummy link, or Gazebo would not take care of root link's inertia -->
   <link name="world"/>
-  <joint name="joint_world_chassis0" type="planar">
+  <joint name="joint_world_log" type="fixed">
+    <origin rpy="0 0 0" xyz="0 0 0"/>
     <parent link="world"/>
-    <child link="link_chassis_0"/>
+    <child link="link_log"/>
+  </joint>
+  <link name="link_log">
+    <visual>
+      <origin rpy="0 ${PI/2} 0" xyz="0 0 0"/>
+      <geometry>
+        <cylinder length="2" radius="0.01"/>
+      </geometry>
+      <material name="red"/>
+    </visual>
+    <collision>
+      <origin rpy="0 ${PI/2} 0" xyz="0 0 0"/>
+      <geometry>
+        <cylinder length="2" radius="0.01"/>
+      </geometry>
+    </collision>
+    <inertial>
+      <mass value="0.1"/>
+      <origin rpy="0 ${PI/2} 0" xyz="0 0 0"/>
+      <inertia ixx="${EPSILON}" ixy="0" ixz="0" iyy="${EPSILON}" iyz="0" izz="${EPSILON}"/>
+    </inertial>
+  </link>
+  <joint name="joint_log_hat0" type="revolute">
+    <origin rpy="0 0 0" xyz="-1 0 0"/>
+    <parent link="link_log"/>
+    <child link="link_hat_0"/>
+    <axis rpy="0 0 0" xyz="0 0 1"/>
+    <limit effort="0" lower="0" upper="0" velocity="0"/>
+  </joint>
+  <link name="link_hat_0">
+    <visual>
+      <origin rpy="0 0 0" xyz="0 0 -0.04"/>
+      <geometry>
+        <cylinder length="0.08" radius="0.02"/>
+      </geometry>
+      <material name="orange"/>
+    </visual>
+    <collision>
+      <origin rpy="0 0 0" xyz="0 0 -0.04"/>
+      <geometry>
+        <cylinder length="0.08" radius="0.02"/>
+      </geometry>
+    </collision>
+    <inertial>
+      <mass value="0.5"/>
+      <origin rpy="0 0 0" xyz="0 0 -0.04"/>
+      <inertia ixx="${EPSILON}" ixy="0" ixz="0" iyy="${EPSILON}" iyz="0" izz="${EPSILON}"/>
+    </inertial>
+  </link>
+  <joint name="joint_hat0_chassis0" type="continuous">
+    <origin rpy="0 0 0" xyz="0.0 0 -0.13"/>
+    <parent link="link_hat_0"/>
+    <child link="link_chassis_0" />
+    <axis rpy="0 0 0" xyz="0 0 1"/>
   </joint>
   <link name="link_chassis_0">
     <visual>
-      <origin rpy="0 0 0" xyz="0 0 0"/>
+      <origin rpy="0 0 ${-PI/2}" xyz="0 0 0"/>
       <geometry>
         <box size="0.4 0.2 0.1"/>
@@ -22,5 +78,5 @@
     </visual>
     <collision>
-      <origin rpy="0 0 0" xyz="0 0 0"/>
+      <origin rpy="0 0 ${-PI/2}" xyz="0 0 0"/>
       <geometry>
         <box size="0.4 0.2 0.1"/>
@@ -29,12 +85,12 @@
     <inertial>
       <mass value="2"/>
-      <origin rpy="0 0 0" xyz="0 0 0"/>
-      <inertia ixx="0.0001" ixy="0" ixz="0" iyy="0.0001" iyz="0" izz="0.0001"/>
+      <origin rpy="0 0 ${-PI/2}" xyz="0 0 0"/>
+      <inertia ixx="${EPSILON}" ixy="0" ixz="0" iyy="${EPSILON}" iyz="0" izz="${EPSILON}"/>
     </inertial>
   </link>
   <joint name="joint_chassis0_caster0" type="fixed">
+    <origin rpy="0 0 0" xyz="0 -0.15 -0.05"/>
     <parent link="link_chassis_0"/>
     <child link="link_caster_0"/>
-    <origin rpy="0 0 0" xyz="0.15 0 -0.05"/>
   </joint>
   <link name="link_caster_0">
@@ -55,117 +111,65 @@
       <mass value="0.1"/>
       <origin rpy="0 0 0" xyz="0 0 0"/>
-      <inertia ixx="0.00001" ixy="0" ixz="0" iyy="0.00001" iyz="0" izz="0.00001"/>
+      <inertia ixx="${EPSILON}" ixy="0" ixz="0" iyy="${EPSILON}" iyz="0" izz="${EPSILON}"/>
     </inertial>
   </link>
   <joint name="joint_chassis0_lwheel0" type="continuous">
-    <origin rpy="0 0 0" xyz="-0.16 0.12 0.01"/>
+    <origin rpy="0 0 0" xyz="0.12 0.16 0.01"/>
+    <parent link="link_chassis_0"/>
     <child link="link_left_wheel_0" />
-    <parent link="link_chassis_0"/>
-    <axis rpy="0 0 0" xyz="0 1 0"/>
+    <axis rpy="0 0 0" xyz="1 0 0"/>
   </joint>
   <link name="link_left_wheel_0">
     <visual>
-      <origin rpy="${PI/2} 0 0" xyz="0 0 0"/>
-      <geometry>
-        <cylinder length="0.04" radius="0.1"/>
-      </geometry>
-      <material name="orange"/>
-    </visual>
-    <collision>
-      <origin rpy="${PI/2} 0 0" xyz="0 0 0" />
-      <geometry>
-        <cylinder length="0.04" radius="0.1"/>
-      </geometry>
-    </collision>
-    <inertial>
-      <mass value="0.5"/>
-      <origin rpy="0 0 0" xyz="0 0 0"/>
-      <inertia ixx="0.0001" ixy="0" ixz="0" iyy="0.0001" iyz="0" izz="0.0001"/>
+      <origin rpy="0 ${PI/2} 0" xyz="0 0 0"/>
+      <geometry>
+        <cylinder length="0.04" radius="0.1"/>
+      </geometry>
+      <material name="orange"/>
+    </visual>
+    <collision>
+      <origin rpy="0 ${PI/2} 0" xyz="0 0 0" />
+      <geometry>
+        <cylinder length="0.04" radius="0.1"/>
+      </geometry>
+    </collision>
+    <inertial>
+      <mass value="0.5"/>
+      <origin rpy="0 ${PI/2} 0" xyz="0 0 0"/>
+      <inertia ixx="${EPSILON}" ixy="0" ixz="0" iyy="${EPSILON}" iyz="0" izz="${EPSILON}"/>
     </inertial>
   </link>
   <joint name="joint_chassis0_rwheel0" type="continuous">
-    <origin rpy="0 0 0" xyz="-0.16 -0.12 0.01"/>
+    <origin rpy="0 0 0" xyz="-0.12 0.16 0.01"/>
     <child link="link_right_wheel_0" />
     <parent link="link_chassis_0"/>
-    <axis rpy="0 0 0" xyz="0 1 0"/>
+    <axis rpy="0 0 0" xyz="1 0 0"/>
   </joint>
   <link name="link_right_wheel_0">
     <collision>
-      <origin rpy="${PI/2} 0 0" xyz="0 0 0" />
-      <geometry>
-        <cylinder length="0.04" radius="0.1"/>
-      </geometry>
-    </collision>
-    <visual>
-      <origin rpy="${PI/2} 0 0" xyz="0 0 0"/>
-      <geometry>
-        <cylinder length="0.04" radius="0.1"/>
-      </geometry>
-      <material name="orange"/>
-    </visual>
-    <inertial>
-      <mass value="0.5"/>
-      <origin rpy="0 0 0" xyz="0 0 0"/>
-      <inertia ixx="0.0001" ixy="0" ixz="0" iyy="0.0001" iyz="0" izz="0.0001"/>
-    </inertial>
-  </link>
-  <joint name="joint_chassis0_hat0" type="revolute">
-    <origin rpy="0 0 0" xyz="0.0 0 0.09"/>
-    <limit effort="0" lower="0" upper="0" velocity="0"/>
-    <child link="link_hat_0" />
-    <parent link="link_chassis_0"/>
-    <axis rpy="0 0 0" xyz="0 0 1"/>
-  </joint>
-  <link name="link_hat_0">
-    <visual>
-      <origin rpy="0 0 0" xyz="0 0 0"/>
-      <geometry>
-        <cylinder length="0.08" radius="0.02"/>
-      </geometry>
-      <material name="orange"/>
-    </visual>
-    <collision>
-      <origin rpy="0 0 0" xyz="0 0 0"/>
-      <geometry>
-        <cylinder length="0.08" radius="0.02"/>
-      </geometry>
-    </collision>
-    <inertial>
-      <mass value="0.5"/>
-      <origin rpy="0 0 0" xyz="0 0 0"/>
-      <inertia ixx="0.00001" ixy="0" ixz="0" iyy="0.00001" iyz="0" izz="0.00001"/>
-    </inertial>
-  </link>
-  <joint name="joint_hat0_log" type="continuous">
-    <parent link="link_hat_0"/>
-    <child link="link_log"/>
-    <origin rpy="0 0 0" xyz="0 0 0.04"/>
-    <axis rpy="0 0 0" xyz="0 0 1"/>
-  </joint>
-  <link name="link_log">
-    <visual>
-      <origin rpy="${PI/2} 0 0" xyz="0 1 0"/>
-      <geometry>
-        <cylinder length="2" radius="0.01"/>
-      </geometry>
-      <material name="red"/>
-    </visual>
-    <collision>
-      <origin rpy="${PI/2} 0 0" xyz="0 1 0"/>
-      <geometry>
-        <cylinder length="2" radius="0.01"/>
-      </geometry>
-    </collision>
-    <inertial>
-      <mass value="0.5"/>
-      <origin rpy="${PI/2} 0 0" xyz="0 1 0"/>
-      <inertia ixx="0.00001" ixy="0" ixz="0" iyy="0.00001" iyz="0" izz="0.00001"/>
-    </inertial>
-  </link>
-  <joint name="joint_log_hat1" type="continuous">
+      <origin rpy="0 ${PI/2} 0" xyz="0 0 0" />
+      <geometry>
+        <cylinder length="0.04" radius="0.1"/>
+      </geometry>
+    </collision>
+    <visual>
+      <origin rpy="0 ${PI/2} 0" xyz="0 0 0"/>
+      <geometry>
+        <cylinder length="0.04" radius="0.1"/>
+      </geometry>
+      <material name="orange"/>
+    </visual>
+    <inertial>
+      <mass value="0.5"/>
+      <origin rpy="0 ${PI/2} 0" xyz="0 0 0"/>
+      <inertia ixx="${EPSILON}" ixy="0" ixz="0" iyy="${EPSILON}" iyz="0" izz="${EPSILON}"/>
+    </inertial>
+  </link>
+  <joint name="joint_log_hat1" type="revolute">
+    <origin rpy="0 0 0" xyz="1 0 0"/>
     <parent link="link_log"/>
     <child link="link_hat_1"/>
-    <origin rpy="0 0 0" xyz="0 2 0"/>
     <axis rpy="0 0 0" xyz="0 0 1"/>
+    <limit effort="0" lower="0" upper="0" velocity="0"/>
   </joint>
   <link name="link_hat_1">
@@ -186,23 +190,23 @@
       <mass value="0.5"/>
       <origin rpy="0 0 0" xyz="0 0 -0.04"/>
-      <inertia ixx="0.00001" ixy="0" ixz="0" iyy="0.00001" iyz="0" izz="0.00001"/>
-    </inertial>
-  </link>
-  <joint name="joint_hat1_chassis1" type="revolute">
+      <inertia ixx="${EPSILON}" ixy="0" ixz="0" iyy="${EPSILON}" iyz="0" izz="${EPSILON}"/>
+    </inertial>
+  </link>
+  <joint name="joint_hat1_chassis1" type="continuous">
     <origin rpy="0 0 0" xyz="0.0 0 -0.13"/>
-    <limit effort="0" lower="0" upper="0" velocity="0"/>
-    <parent link="link_hat_1" />
-    <child link="link_chassis_1"/>
+    <parent link="link_hat_1"/>
+    <child link="link_chassis_1" />
+    <axis rpy="0 0 0" xyz="0 0 1"/>
   </joint>
   <link name="link_chassis_1">
     <visual>
-      <origin rpy="0 0 0" xyz="0 0 0"/>
+      <origin rpy="0 0 ${-PI/2}" xyz="0 0 0"/>
       <geometry>
         <box size="0.4 0.2 0.1"/>
       </geometry>
-      <material name="black"/>
-    </visual>
-    <collision>
-      <origin rpy="0 0 0" xyz="0 0 0"/>
+      <material name="white"/>
+    </visual>
+    <collision>
+      <origin rpy="0 0 ${-PI/2}" xyz="0 0 0"/>
       <geometry>
         <box size="0.4 0.2 0.1"/>
@@ -211,12 +215,12 @@
     <inertial>
       <mass value="2"/>
-      <origin rpy="0 0 0" xyz="0 0 0"/>
-      <inertia ixx="0.0001" ixy="0" ixz="0" iyy="0.0001" iyz="0" izz="0.0001"/>
+      <origin rpy="0 0 ${-PI/2}" xyz="0 0 0"/>
+      <inertia ixx="${EPSILON}" ixy="0" ixz="0" iyy="${EPSILON}" iyz="0" izz="${EPSILON}"/>
     </inertial>
   </link>
   <joint name="joint_chassis1_caster1" type="fixed">
+    <origin rpy="0 0 0" xyz="0 -0.15 -0.05"/>
     <parent link="link_chassis_1"/>
     <child link="link_caster_1"/>
-    <origin rpy="0 0 0" xyz="0.15 0 -0.05"/>
   </joint>
   <link name="link_caster_1">
@@ -237,58 +241,188 @@
       <mass value="0.1"/>
       <origin rpy="0 0 0" xyz="0 0 0"/>
-      <inertia ixx="0.00001" ixy="0" ixz="0" iyy="0.00001" iyz="0" izz="0.00001"/>
+      <inertia ixx="${EPSILON}" ixy="0" ixz="0" iyy="${EPSILON}" iyz="0" izz="${EPSILON}"/>
     </inertial>
   </link>
   <joint name="joint_chassis1_lwheel1" type="continuous">
-    <origin rpy="0 0 0" xyz="-0.16 0.12 0.01"/>
+    <origin rpy="0 0 0" xyz="0.12 0.16 0.01"/>
+    <parent link="link_chassis_1"/>
     <child link="link_left_wheel_1" />
-    <parent link="link_chassis_1"/>
-    <axis rpy="0 0 0" xyz="0 1 0"/>
+    <axis rpy="0 0 0" xyz="1 0 0"/>
   </joint>
   <link name="link_left_wheel_1">
     <visual>
-      <origin rpy="${PI/2} 0 0" xyz="0 0 0"/>
-      <geometry>
-        <cylinder length="0.04" radius="0.1"/>
-      </geometry>
-      <material name="orange"/>
-    </visual>
-    <collision>
-      <origin rpy="${PI/2} 0 0" xyz="0 0 0" />
-      <geometry>
-        <cylinder length="0.04" radius="0.1"/>
-      </geometry>
-    </collision>
-    <inertial>
-      <mass value="0.5"/>
-      <origin rpy="0 0 0" xyz="0 0 0"/>
-      <inertia ixx="0.0001" ixy="0" ixz="0" iyy="0.0001" iyz="0" izz="0.0001"/>
+      <origin rpy="0 ${PI/2} 0" xyz="0 0 0"/>
+      <geometry>
+        <cylinder length="0.04" radius="0.1"/>
+      </geometry>
+      <material name="orange"/>
+    </visual>
+    <collision>
+      <origin rpy="0 ${PI/2} 0" xyz="0 0 0" />
+      <geometry>
+        <cylinder length="0.04" radius="0.1"/>
+      </geometry>
+    </collision>
+    <inertial>
+      <mass value="0.5"/>
+      <origin rpy="0 ${PI/2} 0" xyz="0 0 0"/>
+      <inertia ixx="${EPSILON}" ixy="0" ixz="0" iyy="${EPSILON}" iyz="0" izz="${EPSILON}"/>
     </inertial>
   </link>
   <joint name="joint_chassis1_rwheel1" type="continuous">
-    <origin rpy="0 0 0" xyz="-0.16 -0.12 0.01"/>
+    <origin rpy="0 0 0" xyz="-0.12 0.16 0.01"/>
     <child link="link_right_wheel_1" />
     <parent link="link_chassis_1"/>
-    <axis rpy="0 0 0" xyz="0 1 0"/>
+    <axis rpy="0 0 0" xyz="1 0 0"/>
   </joint>
   <link name="link_right_wheel_1">
     <collision>
-      <origin rpy="${PI/2} 0 0" xyz="0 0 0" />
-      <geometry>
-        <cylinder length="0.04" radius="0.1"/>
-      </geometry>
-    </collision>
-    <visual>
-      <origin rpy="${PI/2} 0 0" xyz="0 0 0"/>
-      <geometry>
-        <cylinder length="0.04" radius="0.1"/>
-      </geometry>
-      <material name="orange"/>
-    </visual>
-    <inertial>
-      <mass value="0.5"/>
-      <origin rpy="0 0 0" xyz="0 0 0"/>
-      <inertia ixx="0.0001" ixy="0" ixz="0" iyy="0.0001" iyz="0" izz="0.0001"/>
-    </inertial>
-  </link>
+      <origin rpy="0 ${PI/2} 0" xyz="0 0 0" />
+      <geometry>
+        <cylinder length="0.04" radius="0.1"/>
+      </geometry>
+    </collision>
+    <visual>
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