Commit message: update two loggers model, use round chassis

File: loggers_description/urdf/two_loggers.urdf.xacro (robot description, xacro)
@@ -16,4 +16,11 @@
   <xacro:property name="L_CHASSIS" value="0.1"/>
   <xacro:property name="M_CHASSIS" value="2"/>
+  <!-- properties of link_caster* -->
+  <xacro:property name="R_CASTER" value="0.04"/>
+  <xacro:property name="M_CASTER" value="0.1"/>
+  <!-- properties of link_wheel* -->
+  <xacro:property name="R_WHEEL" value="0.09"/>
+  <xacro:property name="L_WHEEL" value="0.04"/>
+  <xacro:property name="M_WHEEL" value="0.5"/>
   <!-- Import all Gazebo-customization elements, including Gazebo colors -->
   <xacro:include filename="$(find loggers_description)/urdf/two_loggers.gazebo" />
@@ -32,5 +39,5 @@
         <cylinder length="${L_LOG}" radius="${R_LOG}"/>
       </geometry>
-      <material name="red"/>
+p      <material name="red"/>
     </visual>
     <collision>
@@ -99,210 +106,210 @@
     </inertial>
   </link>
-  <!-- <joint name="joint_chassis0_caster0" type="fixed"> -->
-  <!--   <origin rpy="0 0 0" xyz="0 -0.15 -0.05"/> -->
-  <!--   <parent link="link_chassis_0"/> -->
-  <!--   <child link="link_caster_0"/> -->
-  <!-- </joint> -->
-  <!-- <link name="link_caster_0"> -->
-  <!--   <visual> -->
-  <!--     <origin rpy="0 0 0" xyz="0 0 0"/> -->
-  <!--     <geometry> -->
-  <!--       <sphere radius="0.04"/> -->
-  <!--     </geometry> -->
-  <!--     <material name="grey"/> -->
-  <!--   </visual> -->
-  <!--   <collision> -->
-  <!--     <origin rpy=" 0 0 0" xyz="0 0 0"/> -->
-  <!--     <geometry> -->
-  <!--       <sphere radius="0.04"/> -->
-  <!--     </geometry> -->
-  <!--   </collision> -->
-  <!--   <inertial> -->
-  <!--     <mass value="0.1"/> -->
-  <!--     <origin rpy="0 0 0" xyz="0 0 0"/> -->
-  <!--     <inertia ixx="${EPSILON}" ixy="0" ixz="0" iyy="${EPSILON}" iyz="0" izz="${EPSILON}"/> -->
-  <!--   </inertial> -->
-  <!-- </link> -->
-  <!-- <joint name="joint_chassis0_lwheel0" type="continuous"> -->
-  <!--   <origin rpy="0 0 0" xyz="0.12 0.16 0.01"/> -->
-  <!--   <parent link="link_chassis_0"/> -->
-  <!--   <child link="link_left_wheel_0" /> -->
-  <!--   <axis rpy="0 0 0" xyz="1 0 0"/> -->
-  <!-- </joint> -->
-  <!-- <link name="link_left_wheel_0"> -->
-  <!--   <visual> -->
-  <!--     <origin rpy="0 ${PI/2} 0" xyz="0 0 0"/> -->
-  <!--     <geometry> -->
-  <!--       <cylinder length="0.04" radius="0.1"/> -->
-  <!--     </geometry> -->
-  <!--     <material name="orange"/> -->
-  <!--   </visual> -->
-  <!--   <collision> -->
-  <!--     <origin rpy="0 ${PI/2} 0" xyz="0 0 0" /> -->
-  <!--     <geometry> -->
-  <!--       <cylinder length="0.04" radius="0.1"/> -->
-  <!--     </geometry> -->
-  <!--   </collision> -->
-  <!--   <inertial> -->
-  <!--     <mass value="0.5"/> -->
-  <!--     <origin rpy="0 ${PI/2} 0" xyz="0 0 0"/> -->
-  <!--     <inertia ixx="${EPSILON}" ixy="0" ixz="0" iyy="${EPSILON}" iyz="0" izz="${EPSILON}"/> -->
-  <!--   </inertial> -->
-  <!-- </link> -->
-  <!-- <joint name="joint_chassis0_rwheel0" type="continuous"> -->
-  <!--   <origin rpy="0 0 0" xyz="-0.12 0.16 0.01"/> -->
-  <!--   <child link="link_right_wheel_0" /> -->
-  <!--   <parent link="link_chassis_0"/> -->
-  <!--   <axis rpy="0 0 0" xyz="1 0 0"/> -->
-  <!-- </joint> -->
-  <!-- <link name="link_right_wheel_0"> -->
-  <!--   <collision> -->
-  <!--     <origin rpy="0 ${PI/2} 0" xyz="0 0 0" /> -->
-  <!--     <geometry> -->
-  <!--       <cylinder length="0.04" radius="0.1"/> -->
-  <!--     </geometry> -->
-  <!--   </collision> -->
-  <!--   <visual> -->
-  <!--     <origin rpy="0 ${PI/2} 0" xyz="0 0 0"/> -->
-  <!--     <geometry> -->
-  <!--       <cylinder length="0.04" radius="0.1"/> -->
-  <!--     </geometry> -->
-  <!--     <material name="orange"/> -->
-  <!--   </visual> -->
-  <!--   <inertial> -->
-  <!--     <mass value="0.5"/> -->
-  <!--     <origin rpy="0 ${PI/2} 0" xyz="0 0 0"/> -->
-  <!--     <inertia ixx="${EPSILON}" ixy="0" ixz="0" iyy="${EPSILON}" iyz="0" izz="${EPSILON}"/> -->
-  <!--   </inertial> -->
-  <!-- </link> -->
-  <!-- <joint name="joint_log_hat1" type="revolute"> -->
-  <!--   <origin rpy="0 0 0" xyz="1 0 0"/> -->
-  <!--   <parent link="link_log"/> -->
-  <!--   <child link="link_hat_1"/> -->
-  <!--   <axis rpy="0 0 0" xyz="0 0 1"/> -->
-  <!--   <limit effort="0" lower="0" upper="0" velocity="0"/> -->
-  <!-- </joint> -->
-  <!-- <link name="link_hat_1"> -->
-  <!--   <visual> -->
-  <!--     <origin rpy="0 0 0" xyz="0 0 -0.04"/> -->
-  <!--     <geometry> -->
-  <!--       <cylinder length="0.08" radius="0.02"/> -->
-  <!--     </geometry> -->
-  <!--     <material name="orange"/> -->
-  <!--   </visual> -->
-  <!--   <collision> -->
-  <!--     <origin rpy="0 0 0" xyz="0 0 -0.04"/> -->
-  <!--     <geometry> -->
-  <!--       <cylinder length="0.08" radius="0.02"/> -->
-  <!--     </geometry> -->
-  <!--   </collision> -->
-  <!--   <inertial> -->
-  <!--     <mass value="0.5"/> -->
-  <!--     <origin rpy="0 0 0" xyz="0 0 -0.04"/> -->
-  <!--     <inertia ixx="${EPSILON}" ixy="0" ixz="0" iyy="${EPSILON}" iyz="0" izz="${EPSILON}"/> -->
-  <!--   </inertial> -->
-  <!-- </link> -->
-  <!-- <joint name="joint_hat1_chassis1" type="continuous"> -->
-  <!--   <origin rpy="0 0 0" xyz="0.0 0 -0.13"/> -->
-  <!--   <parent link="link_hat_1"/> -->
-  <!--   <child link="link_chassis_1" /> -->
-  <!--   <axis rpy="0 0 0" xyz="0 0 1"/> -->
-  <!-- </joint> -->
-  <!-- <link name="link_chassis_1"> -->
-  <!--   <visual> -->
-  <!--     <origin rpy="0 0 ${-PI/2}" xyz="0 0 0"/> -->
-  <!--     <geometry> -->
-  <!--       <box size="0.4 0.2 0.1"/> -->
-  <!--     </geometry> -->
-  <!--     <material name="white"/> -->
-  <!--   </visual> -->
-  <!--   <collision> -->
-  <!--     <origin rpy="0 0 ${-PI/2}" xyz="0 0 0"/> -->
-  <!--     <geometry> -->
-  <!--       <box size="0.4 0.2 0.1"/> -->
-  <!--     </geometry> -->
-  <!--   </collision> -->
-  <!--   <inertial> -->
-  <!--     <mass value="2"/> -->
-  <!--     <origin rpy="0 0 ${-PI/2}" xyz="0 0 0"/> -->
-  <!--     <inertia ixx="${EPSILON}" ixy="0" ixz="0" iyy="${EPSILON}" iyz="0" izz="${EPSILON}"/> -->
-  <!--   </inertial> -->
-  <!-- </link> -->
-  <!-- <joint name="joint_chassis1_caster1" type="fixed"> -->
-  <!--   <origin rpy="0 0 0" xyz="0 -0.15 -0.05"/> -->
-  <!--   <parent link="link_chassis_1"/> -->
-  <!--   <child link="link_caster_1"/> -->
-  <!-- </joint> -->
-  <!-- <link name="link_caster_1"> -->
-  <!--   <visual> -->
-  <!--     <origin rpy="0 0 0" xyz="0 0 0"/> -->
-  <!--     <geometry> -->
-  <!--       <sphere radius="0.04"/> -->
-  <!--     </geometry> -->
-  <!--     <material name="grey"/> -->
-  <!--   </visual> -->
-  <!--   <collision> -->
-  <!--     <origin rpy=" 0 0 0" xyz="0 0 0"/> -->
-  <!--     <geometry> -->
-  <!--       <sphere radius="0.04"/> -->
-  <!--     </geometry> -->
-  <!--   </collision> -->
-  <!--   <inertial> -->
-  <!--     <mass value="0.1"/> -->
-  <!--     <origin rpy="0 0 0" xyz="0 0 0"/> -->
-  <!--     <inertia ixx="${EPSILON}" ixy="0" ixz="0" iyy="${EPSILON}" iyz="0" izz="${EPSILON}"/> -->
-  <!--   </inertial> -->
-  <!-- </link> -->
-  <!-- <joint name="joint_chassis1_lwheel1" type="continuous"> -->
-  <!--   <origin rpy="0 0 0" xyz="0.12 0.16 0.01"/> -->
-  <!--   <parent link="link_chassis_1"/> -->
-  <!--   <child link="link_left_wheel_1" /> -->
-  <!--   <axis rpy="0 0 0" xyz="1 0 0"/> -->
-  <!-- </joint> -->
-  <!-- <link name="link_left_wheel_1"> -->
-  <!--   <visual> -->
-  <!--     <origin rpy="0 ${PI/2} 0" xyz="0 0 0"/> -->
-  <!--     <geometry> -->
-  <!--       <cylinder length="0.04" radius="0.1"/> -->
-  <!--     </geometry> -->
-  <!--     <material name="orange"/> -->
-  <!--   </visual> -->
-  <!--   <collision>  -->
-  <!--     <origin rpy="0 ${PI/2} 0" xyz="0 0 0" /> -->
-  <!--     <geometry> -->
-  <!--       <cylinder length="0.04" radius="0.1"/> -->
-  <!--     </geometry> -->
-  <!--   </collision> -->
-  <!--   <inertial> -->
-  <!--     <mass value="0.5"/> -->
-  <!--     <origin rpy="0 ${PI/2} 0" xyz="0 0 0"/> -->
-  <!--     <inertia ixx="${EPSILON}" ixy="0" ixz="0" iyy="${EPSILON}" iyz="0" izz="${EPSILON}"/> -->
-  <!--   </inertial> -->
-  <!-- </link> -->
-  <!-- <joint name="joint_chassis1_rwheel1" type="continuous"> -->
-  <!--   <origin rpy="0 0 0" xyz="-0.12 0.16 0.01"/> -->
-  <!--   <child link="link_right_wheel_1" /> -->
-  <!--   <parent link="link_chassis_1"/> -->
-  <!--   <axis rpy="0 0 0" xyz="1 0 0"/> -->
-  <!-- </joint> -->
-  <!-- <link name="link_right_wheel_1"> -->
-  <!--   <collision> -->
-  <!--     <origin rpy="0 ${PI/2} 0" xyz="0 0 0" /> -->
-  <!--     <geometry> -->
-  <!--       <cylinder length="0.04" radius="0.1"/> -->
-  <!--     </geometry> -->
-  <!--   </collision> -->
-  <!--   <visual> -->
-  <!--     <origin rpy="0 ${PI/2} 0" xyz="0 0 0"/> -->
-  <!--     <geometry> -->
-  <!--       <cylinder length="0.04" radius="0.1"/> -->
-  <!--     </geometry> -->
-  <!--     <material name="orange"/> -->
-  <!--   </visual> -->
-  <!--   <inertial> -->
-  <!--     <mass value="0.5"/> -->
-  <!--     <origin rpy="0 ${PI/2} 0" xyz="0 0 0"/> -->
-  <!--     <inertia ixx="${EPSILON}" ixy="0" ixz="0" iyy="${EPSILON}" iyz="0" izz="${EPSILON}"/> -->
-  <!--   </inertial> -->
-  <!-- </link> -->
+  <joint name="joint_chassis0_caster0" type="fixed">
+    <origin rpy="0 0 0" xyz="0 ${-R_CHASSIS/2} ${-L_CHASSIS/2}"/>
+    <parent link="link_chassis_0"/>
+    <child link="link_caster_0"/>
+  </joint>
+  <link name="link_caster_0">
+    <visual>
+      <origin rpy="0 0 0" xyz="0 0 0"/>
+      <geometry>
+        <sphere radius="${R_CASTER}"/>
+      </geometry>
+      <material name="grey"/>
+    </visual>
+    <collision>
+      <origin rpy=" 0 0 0" xyz="0 0 0"/>
+      <geometry>
+        <sphere radius="${R_CASTER}"/>
+      </geometry>
+    </collision>
+    <inertial>
+      <mass value="${M_CASTER}"/>
+      <origin rpy="0 0 0" xyz="0 0 0"/>
+      <inertia ixx="${2/5*M_CASTER*R_CASTER*R_CASTER}" ixy="0" ixz="0" iyy="${2/5*M_CASTER*R_CASTER*R_CASTER}" iyz="0" izz="${2/5*M_CASTER*R_CASTER*R_CASTER}"/>
+    </inertial>
+  </link>
+  <joint name="joint_chassis0_lwheel0" type="continuous">
+    <origin rpy="0 0 0" xyz="${R_CHASSIS/2} ${R_CHASSIS/2} 0"/>
+    <parent link="link_chassis_0"/>
+    <child link="link_left_wheel_0" />
+    <axis rpy="0 0 0" xyz="1 0 0"/>
+  </joint>
+  <link name="link_left_wheel_0">
+    <visual>
+      <origin rpy="0 ${PI/2} 0" xyz="0 0 0"/>
+      <geometry>
+        <cylinder length="${L_WHEEL}" radius="${R_WHEEL}"/>
+      </geometry>
+      <material name="orange"/>
+    </visual>
+    <collision>
+      <origin rpy="0 ${PI/2} 0" xyz="0 0 0" />
+      <geometry>
+        <cylinder length="${L_WHEEL}" radius="${R_WHEEL}"/>
+      </geometry>
+    </collision>
+    <inertial>
+      <mass value="${M_WHEEL}"/>
+      <origin rpy="0 ${PI/2} 0" xyz="0 0 0"/>
+      <inertia ixx="${1/12*M_WHEEL*(3*R_WHEEL*R_WHEEL+L_WHEEL*L_WHEEL)}" ixy="0" ixz="0" iyy="${1/12*M_WHEEL*(3*R_WHEEL*R_WHEEL+L_WHEEL*L_WHEEL)}" iyz="0" izz="${1/2*M_WHEEL*R_WHEEL*R_WHEEL}"/>
+    </inertial>
+  </link>
+  <joint name="joint_chassis0_rwheel0" type="continuous">
+    <origin rpy="0 0 0" xyz="${-R_CHASSIS/2} ${R_CHASSIS/2} 0"/>
+    <child link="link_right_wheel_0" />
+    <parent link="link_chassis_0"/>
+    <axis rpy="0 0 0" xyz="1 0 0"/>
+  </joint>
+  <link name="link_right_wheel_0">
+    <collision>
+      <origin rpy="0 ${PI/2} 0" xyz="0 0 0" />
+      <geometry>
+        <cylinder length="${L_WHEEL}" radius="${R_WHEEL}"/>
+      </geometry>
+    </collision>
+    <visual>
+      <origin rpy="0 ${PI/2} 0" xyz="0 0 0"/>
+      <geometry>
+        <cylinder length="${L_WHEEL}" radius="${R_WHEEL}"/>
+      </geometry>
+      <material name="orange"/>
+    </visual>
+    <inertial>
+      <mass value="${M_WHEEL}"/>
+      <origin rpy="0 ${PI/2} 0" xyz="0 0 0"/>
+      <inertia ixx="${1/12*M_WHEEL*(3*R_WHEEL*R_WHEEL+L_WHEEL*L_WHEEL)}" ixy="0" ixz="0" iyy="${1/12*M_WHEEL*(3*R_WHEEL*R_WHEEL+L_WHEEL*L_WHEEL)}" iyz="0" izz="${1/2*M_WHEEL*R_WHEEL*R_WHEEL}"/>
+    </inertial>
+  </link>
+  <joint name="joint_log_hat1" type="revolute">
+    <origin rpy="0 0 0" xyz="${L_LOG/2} 0 0"/>
+    <parent link="link_log"/>
+    <child link="link_hat_1"/>
+    <axis rpy="0 0 0" xyz="0 0 1"/>
+    <limit effort="0" lower="0" upper="0" velocity="0"/>
+  </joint>
+  <link name="link_hat_1">
+    <visual>
+      <origin rpy="0 0 0" xyz="0 0 ${-L_HAT/2}"/>
+      <geometry>
+        <cylinder length="${L_HAT}" radius="${R_HAT}"/>
+      </geometry>
+      <material name="orange"/>
+    </visual>
+    <collision>
+      <origin rpy="0 0 0" xyz="0 0 ${-L_HAT/2}"/>
+      <geometry>
+        <cylinder length="${L_HAT}" radius="${R_HAT}"/>
+      </geometry>
+    </collision>
+    <inertial>
+      <mass value="${M_HAT}"/>
+      <origin rpy="0 0 0" xyz="0 0 ${-L_HAT/2}"/>
+      <inertia ixx="${1/12*M_HAT*(3*R_HAT*R_HAT+L_HAT*L_HAT)}" ixy="0" ixz="0" iyy="${1/12*M_HAT*(3*R_HAT*R_HAT+L_HAT*L_HAT)}" iyz="0" izz="${1/2*M_HAT*R_HAT*R_HAT}"/>
+    </inertial>
+  </link>
+  <joint name="joint_hat1_chassis1" type="continuous">
+    <origin rpy="0 0 0" xyz="0.0 0 ${-L_HAT-L_CHASSIS/2}"/>
+    <parent link="link_hat_1"/>
+    <child link="link_chassis_1" />
+    <axis rpy="0 0 0" xyz="0 0 1"/>
+  </joint>
+  <link name="link_chassis_1">
+    <visual>
+      <origin rpy="0 0 0" xyz="0 0 0"/>
+      <geometry>
+        <cylinder length="${L_CHASSIS}" radius="${R_CHASSIS}"/>
+      </geometry>
+      <material name="black"/>
+    </visual>
+    <collision>
+      <origin rpy="0 0 0" xyz="0 0 0"/>
+      <geometry>
+        <cylinder length="${L_CHASSIS}" radius="${R_CHASSIS}"/>
+      </geometry>
+    </collision>
+    <inertial>
+      <mass value="2"/>
+      <origin rpy="0 0 0" xyz="0 0 0"/>
+      <inertia ixx="${1/12*M_CHASSIS*(3*R_CHASSIS*R_CHASSIS+L_CHASSIS*L_CHASSIS)}" ixy="0" ixz="0" iyy="${1/12*M_CHASSIS*(3*R_CHASSIS*R_CHASSIS+L_CHASSIS*L_CHASSIS)}" iyz="0" izz="${1/2*M_CHASSIS*R_CHASSIS*R_CHASSIS}"/>
+    </inertial>
+  </link>
+  <joint name="joint_chassis1_caster1" type="fixed">
+    <origin rpy="0 0 0" xyz="0 ${-R_CHASSIS/2} ${-L_CHASSIS/2}"/>
+    <parent link="link_chassis_1"/>
+    <child link="link_caster_1"/>
+  </joint>
+  <link name="link_caster_1">
+    <visual>
+      <origin rpy="0 0 0" xyz="0 0 0"/>
+      <geometry>
+        <sphere radius="${R_CASTER}"/>
+      </geometry>
+      <material name="grey"/>
+    </visual>
+    <collision>
+      <origin rpy=" 0 0 0" xyz="0 0 0"/>
+      <geometry>
+        <sphere radius="${R_CASTER}"/>
+      </geometry>
+    </collision>
+    <inertial>
+      <mass value="${M_CASTER}"/>
+      <origin rpy="0 0 0" xyz="0 0 0"/>
+      <inertia ixx="${2/5*M_CASTER*R_CASTER*R_CASTER}" ixy="0" ixz="0" iyy="${2/5*M_CASTER*R_CASTER*R_CASTER}" iyz="0" izz="${2/5*M_CASTER*R_CASTER*R_CASTER}"/>
+    </inertial>
+  </link>
+  <joint name="joint_chassi10_lwheel1" type="continuous">
+    <origin rpy="0 0 0" xyz="${R_CHASSIS/2} ${R_CHASSIS/2} 0"/>
+    <parent link="link_chassis_1"/>
+    <child link="link_left_wheel_1" />
+    <axis rpy="0 0 0" xyz="1 0 0"/>
+  </joint>
+  <link name="link_left_wheel_1">
+    <visual>
+      <origin rpy="0 ${PI/2} 0" xyz="0 0 0"/>
+      <geometry>
+        <cylinder length="${L_WHEEL}" radius="${R_WHEEL}"/>
+      </geometry>
+      <material name="orange"/>
+    </visual>
+    <collision>
+      <origin rpy="0 ${PI/2} 0" xyz="0 0 0" />
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
Commit message: fix /cmd_vel_0 and /cmd_vel_1 in two loggers

File: loggers_description/urdf/two_loggers.urdf.xacro (robot description, xacro)
@@ -261,5 +261,5 @@
     </inertial>
   </link>
-  <joint name="joint_chassi10_lwheel1" type="continuous">
+  <joint name="joint_chassis1_lwheel1" type="continuous">
     <origin rpy="0 0 0" xyz="${R_CHASSIS/2} ${R_CHASSIS/2} 0"/>
     <parent link="link_chassis_1"/>

Commit message: add joint damping to two_loggers urdf

File: loggers_description/urdf/two_loggers.urdf.xacro (robot description, xacro)
@@ -59,4 +59,5 @@
     <axis rpy="0 0 0" xyz="0 0 1"/>
     <limit effort="0" lower="0" upper="0" velocity="0"/>
+    <dynamics damping="0.1" friction="0.0"/>
   </joint>
   <link name="link_hat_0">
@@ -85,4 +86,5 @@
     <child link="link_chassis_0" />
     <axis rpy="0 0 0" xyz="0 0 1"/>
+    <dynamics damping="0.1" friction="0.0"/>
   </joint>
   <link name="link_chassis_0">
@@ -110,4 +112,5 @@
     <parent link="link_chassis_0"/>
     <child link="link_caster_0"/>
+    <dynamics damping="0.1" friction="0.0"/>
   </joint>
   <link name="link_caster_0">
@@ -136,4 +139,5 @@
     <child link="link_left_wheel_0" />
     <axis rpy="0 0 0" xyz="1 0 0"/>
+    <dynamics damping="0.1" friction="0.0"/>
   </joint>
   <link name="link_left_wheel_0">
@@ -162,4 +166,5 @@
     <parent link="link_chassis_0"/>
     <axis rpy="0 0 0" xyz="1 0 0"/>
+    <dynamics damping="0.1" friction="0.0"/>
   </joint>
   <link name="link_right_wheel_0">
@@ -189,4 +194,5 @@
     <axis rpy="0 0 0" xyz="0 0 1"/>
     <limit effort="0" lower="0" upper="0" velocity="0"/>
+    <dynamics damping="0.1" friction="0.0"/>
   </joint>
   <link name="link_hat_1">
@@ -215,4 +221,5 @@
     <child link="link_chassis_1" />
     <axis rpy="0 0 0" xyz="0 0 1"/>
+    <dynamics damping="0.1" friction="0.0"/>
   </joint>
   <link name="link_chassis_1">
@@ -240,4 +247,5 @@
     <parent link="link_chassis_1"/>
     <child link="link_caster_1"/>
+    <dynamics damping="0.1" friction="0.0"/>
   </joint>
   <link name="link_caster_1">
@@ -266,4 +274,5 @@
     <child link="link_left_wheel_1" />
     <axis rpy="0 0 0" xyz="1 0 0"/>
+    <dynamics damping="0.1" friction="0.0"/>
   </joint>
   <link name="link_left_wheel_1">
@@ -292,4 +301,5 @@
     <parent link="link_chassis_1"/>
     <axis rpy="0 0 0" xyz="1 0 0"/>
+    <dynamics damping="0.1" friction="0.0"/>
   </joint>
   <link name="link_right_wheel_1">

Commit message: disable damping

File: loggers_description/urdf/two_loggers.urdf.xacro (robot description, xacro)
@@ -4,4 +4,6 @@
   <!-- Constants for robot dimensions -->
   <xacro:property name="PI" value="3.1415926535897931"/>
+  <!-- properties of joint damping* -->
+  <xacro:property name="DAMP" value="0.9"/>
   <!-- properties of link_log -->
   <xacro:property name="R_LOG" value="0.01"/>
@@ -59,5 +61,4 @@
     <axis rpy="0 0 0" xyz="0 0 1"/>
     <limit effort="0" lower="0" upper="0" velocity="0"/>
-    <dynamics damping="0.1" friction="0.0"/>
   </joint>
   <link name="link_hat_0">
@@ -86,5 +87,4 @@
     <child link="link_chassis_0" />
     <axis rpy="0 0 0" xyz="0 0 1"/>
-    <dynamics damping="0.1" friction="0.0"/>
   </joint>
   <link name="link_chassis_0">
@@ -112,5 +112,4 @@
     <parent link="link_chassis_0"/>
     <child link="link_caster_0"/>
-    <dynamics damping="0.1" friction="0.0"/>
   </joint>
   <link name="link_caster_0">
@@ -139,5 +138,4 @@
     <child link="link_left_wheel_0" />
     <axis rpy="0 0 0" xyz="1 0 0"/>
-    <dynamics damping="0.1" friction="0.0"/>
   </joint>
   <link name="link_left_wheel_0">
@@ -166,5 +164,4 @@
     <parent link="link_chassis_0"/>
     <axis rpy="0 0 0" xyz="1 0 0"/>
-    <dynamics damping="0.1" friction="0.0"/>
   </joint>
   <link name="link_right_wheel_0">
@@ -194,5 +191,4 @@
     <axis rpy="0 0 0" xyz="0 0 1"/>
     <limit effort="0" lower="0" upper="0" velocity="0"/>
-    <dynamics damping="0.1" friction="0.0"/>
   </joint>
   <link name="link_hat_1">
@@ -221,5 +217,4 @@
     <child link="link_chassis_1" />
     <axis rpy="0 0 0" xyz="0 0 1"/>
-    <dynamics damping="0.1" friction="0.0"/>
   </joint>
   <link name="link_chassis_1">
@@ -247,5 +242,4 @@
     <parent link="link_chassis_1"/>
     <child link="link_caster_1"/>
-    <dynamics damping="0.1" friction="0.0"/>
   </joint>
   <link name="link_caster_1">
@@ -274,5 +268,4 @@
     <child link="link_left_wheel_1" />
     <axis rpy="0 0 0" xyz="1 0 0"/>
-    <dynamics damping="0.1" friction="0.0"/>
   </joint>
   <link name="link_left_wheel_1">
@@ -301,5 +294,4 @@
     <parent link="link_chassis_1"/>
     <axis rpy="0 0 0" xyz="1 0 0"/>
-    <dynamics damping="0.1" friction="0.0"/>
   </joint>
   <link name="link_right_wheel_1">

Commit message: upgrade double escape env

File: loggers_description/urdf/two_loggers.urdf.xacro (robot description, xacro)
@@ -61,4 +61,5 @@
     <axis rpy="0 0 0" xyz="0 0 1"/>
     <limit effort="0" lower="0" upper="0" velocity="0"/>
+    <dynamics damping="0.2"/>
   </joint>
   <link name="link_hat_0">
@@ -87,4 +88,5 @@
     <child link="link_chassis_0" />
     <axis rpy="0 0 0" xyz="0 0 1"/>
+    <dynamics damping="0.2"/>
   </joint>
   <link name="link_chassis_0">
@@ -191,4 +193,5 @@
     <axis rpy="0 0 0" xyz="0 0 1"/>
     <limit effort="0" lower="0" upper="0" velocity="0"/>
+    <dynamics damping="0.2"/>
   </joint>
   <link name="link_hat_1">
@@ -217,4 +220,5 @@
     <child link="link_chassis_1" />
     <axis rpy="0 0 0" xyz="0 0 1"/>
+    <dynamics damping="0.2"/>
   </joint>
   <link name="link_chassis_1">

Commit message: deprecate useless functions

File: loggers_description/urdf/two_loggers.urdf.xacro (robot description, xacro)
@@ -9,5 +9,5 @@
   <xacro:property name="R_LOG" value="0.01"/>
   <xacro:property name="L_LOG" value="2"/>
-  <xacro:property name="M_LOG" value="0.4"/>
+  <xacro:property name="M_LOG" value="0.04"/>
   <!-- properties of link_hat* -->
   <xacro:property name="R_HAT" value="0.02"/>

Commit message: create new world

File: loggers_description/urdf/two_loggers.urdf.xacro (robot description, xacro)
@@ -7,6 +7,8 @@
   <xacro:property name="DAMP" value="0.9"/>
   <!-- properties of link_log -->
-  <xacro:property name="R_LOG" value="0.01"/>
-  <xacro:property name="L_LOG" value="2"/>
+  <!-- <xacro:property name="R_LOG" value="0.01"/>
+  <xacro:property name="L_LOG" value="2"/> -->
+  <xacro:property name="R_LOG" value="0.04"/>
+  <xacro:property name="L_LOG" value="2.1"/>
   <xacro:property name="M_LOG" value="0.04"/>
   <!-- properties of link_hat* -->

Commit message: mod double dqn train for the new world

File: loggers_description/urdf/two_loggers.urdf.xacro (robot description, xacro)
@@ -9,5 +9,5 @@
   <!-- <xacro:property name="R_LOG" value="0.01"/>
   <xacro:property name="L_LOG" value="2"/> -->
-  <xacro:property name="R_LOG" value="0.04"/>
+  <xacro:property name="R_LOG" value="0.02"/>
   <xacro:property name="L_LOG" value="2.1"/>
   <xacro:property name="M_LOG" value="0.04"/>
