Commit message: pub ros params when launch world

File: loggers_description/urdf/two_loggers.urdf.xacro (robot description, xacro)
@@ -10,5 +10,5 @@
   <xacro:property name="L_LOG" value="2"/> -->
   <xacro:property name="R_LOG" value="0.02"/>
-  <xacro:property name="L_LOG" value="2.1"/>
+  <xacro:property name="L_LOG" value="2"/>
   <xacro:property name="M_LOG" value="0.04"/>
   <!-- properties of link_hat* -->
@@ -17,5 +17,5 @@
   <xacro:property name="M_HAT" value="0.5"/>
   <!-- properties of link_chassis* -->
-  <xacro:property name="R_CHASSIS" value="0.2"/>
+  <xacro:property name="R_CHASSIS" value="0.25"/>
   <xacro:property name="L_CHASSIS" value="0.1"/>
   <xacro:property name="M_CHASSIS" value="2"/>
