Commit message: modify logger urdf follow rrbot tutorial

File: loggers_description/urdf/single_logger.urdf.xacro (robot description, xacro)
@@ -1,45 +1,24 @@
 <?xml version="1.0" ?>
 <robot name="logger" xmlns:xacro="https://www.ros.org/wiki/xacro" >
-  <material name="black">
-    <color rgba="0.0 0.0 0.0 1.0"/>
-  </material>
-  <material name="blue">
-    <color rgba="0.203125 0.23828125 0.28515625 1.0"/>
-  </material>
-  <material name="green">
-    <color rgba="0.0 0.8 0.0 1.0"/>
-  </material>
-  <material name="grey">
-    <color rgba="0.2 0.2 0.2 1.0"/>
-  </material>
-  <material name="orange">
-    <color rgba="1.0 0.423529411765 0.0392156862745 1.0"/>
-  </material>
-  <material name="brown">
-    <color rgba="0.870588235294 0.811764705882 0.764705882353 1.0"/>
-  </material>
-  <material name="red">
-    <color rgba="0.80078125 0.12890625 0.1328125 1.0"/>
-  </material>
-  <material name="white">
-    <color rgba="1.0 1.0 1.0 1.0"/>
-  </material>
-  <gazebo reference="link_chassis">
-    <material>Gazebo/Orange</material>
-  </gazebo>
-  <gazebo reference="link_left_wheel">
-    <material>Gazebo/Blue</material>
-  </gazebo>
-  <gazebo reference="link_right_wheel">
-    <material>Gazebo/Blue</material>
-  </gazebo>
+  <!-- Constants for robot dimensions -->
+  <xacro:property name="PI" value="3.1415926535897931"/>
+  <xacro:property name="mass" value="1" /> <!-- arbitrary value for mass -->
+  <xacro:property name="width" value="0.1" /> <!-- Square dimensions (widthxwidth) of beams -->
+  <xacro:property name="height1" value="2" /> <!-- Link 1 -->
+  <xacro:property name="height2" value="1" /> <!-- Link 2 -->
+  <xacro:property name="height3" value="1" /> <!-- Link 3 -->
+  <xacro:property name="camera_link" value="0.05" /> <!-- Size of square 'camera' box -->
+  <xacro:property name="axel_offset" value="0.05" /> <!-- Space btw top of beam and the each joint -->
+  <!-- Import all Gazebo-customization elements, including Gazebo colors -->
+  <xacro:include filename="$(find loggers_description)/urdf/single_logger.gazebo" />
+  <!-- Import Rviz colors -->
+  <xacro:include filename="$(find loggers_description)/urdf/materials.xacro" />
+  <!-- Used for fixing robot to Gazebo 'base_link' -->
+  <link name="world"/>
+  <joint name="fixed" type="planar">
+    <parent link="world"/>
+    <child link="link_chassis"/>
+  </joint>
   <link name="link_chassis">
-    <!-- pose and inertial -->
-    <pose>0 0 0.1 0 0 0</pose>
-    <inertial>
-      <mass value="5"/>
-      <origin rpy="0 0 0" xyz="0 0 0.1"/>
-      <inertia ixx="0.0395416666667" ixy="0" ixz="0" iyy="0.106208333333" iyz="0" izz="0.106208333333"/>
-    </inertial>
     <collision name="collision_chassis">
       <geometry>
@@ -54,5 +33,15 @@
       <material name="blue"/>
     </visual>
-    <!-- caster front -->
+    <inertial>
+      <mass value="5"/>
+      <origin rpy="0 0 0" xyz="0 0 0.1"/>
+      <inertia ixx="0.0395416666667" ixy="0" ixz="0" iyy="0.106208333333" iyz="0" izz="0.106208333333"/>
+    </inertial>
+  </link>
+  <joint name="caster_joint" type="fixed">
+    <parent link="link_chassis"/>
+    <child link="caster_front"/>
+  </joint>
+  <link name="caster_front">
     <collision name="caster_front_collision">
       <origin rpy=" 0 0 0" xyz="0.35 0 -0.05"/>
@@ -77,6 +66,13 @@
       </geometry>
     </visual>
-    </link>
-  <!-- Create wheel right -->
+  </link>
+  <joint name="joint_right_wheel" type="continuous">
+    <origin rpy="0 0 0" xyz="-0.05 0.15 0"/>
+    <child link="link_right_wheel" />
+    <parent link="link_chassis"/>
+    <axis rpy="0 0 0" xyz="0 1 0"/>
+    <limit effort="10000" velocity="1000"/>
+    <joint_properties damping="1.0" friction="1.0" />
+  </joint>
   <link name="link_right_wheel">
     <inertial>
@@ -99,12 +95,4 @@
   </link>
   <!--   Joint for right wheel  -->
-  <joint name="joint_right_wheel" type="continuous">
-    <origin rpy="0 0 0" xyz="-0.05 0.15 0"/>
-    <child link="link_right_wheel" />
-    <parent link="link_chassis"/>
-    <axis rpy="0 0 0" xyz="0 1 0"/>
-    <limit effort="10000" velocity="1000"/>
-    <joint_properties damping="1.0" friction="1.0" />
-  </joint>
   <!-- Left Wheel link -->
   <link name="link_left_wheel">

Commit message: create loggers gazebo packge

File: loggers_description/urdf/single_logger.urdf.xacro (robot description, xacro)
@@ -3,11 +3,4 @@
   <!-- Constants for robot dimensions -->
   <xacro:property name="PI" value="3.1415926535897931"/>
-  <xacro:property name="mass" value="1" /> <!-- arbitrary value for mass -->
-  <xacro:property name="width" value="0.1" /> <!-- Square dimensions (widthxwidth) of beams -->
-  <xacro:property name="height1" value="2" /> <!-- Link 1 -->
-  <xacro:property name="height2" value="1" /> <!-- Link 2 -->
-  <xacro:property name="height3" value="1" /> <!-- Link 3 -->
-  <xacro:property name="camera_link" value="0.05" /> <!-- Size of square 'camera' box -->
-  <xacro:property name="axel_offset" value="0.05" /> <!-- Space btw top of beam and the each joint -->
   <!-- Import all Gazebo-customization elements, including Gazebo colors -->
   <xacro:include filename="$(find loggers_description)/urdf/single_logger.gazebo" />
@@ -16,5 +9,5 @@
   <!-- Used for fixing robot to Gazebo 'base_link' -->
   <link name="world"/>
-  <joint name="fixed" type="planar">
+  <joint name="joint_world_chassis" type="floating">
     <parent link="world"/>
     <child link="link_chassis"/>
@@ -65,4 +58,5 @@
         <sphere radius="0.05"/>
       </geometry>
+      <material name="black"/>
     </visual>
   </link>
@@ -92,14 +86,16 @@
         <cylinder length="0.04" radius="0.1"/>
       </geometry>
+      <material name="orange"/>
     </visual>
   </link>
-  <!--   Joint for right wheel  -->
-  <!-- Left Wheel link -->
+  <joint name="joint_left_wheel" type="continuous">
+    <origin rpy="0 0 0" xyz="-0.05 -0.15 0"/>
+    <child link="link_left_wheel" />
+    <parent link="link_chassis"/>
+    <axis rpy="0 0 0" xyz="0 1 0"/>
+    <limit effort="10000" velocity="1000"/>
+    <joint_properties damping="1.0" friction="1.0" />
+  </joint>
   <link name="link_left_wheel">
-    <inertial>
-      <mass value="0.2"/>
-      <origin rpy="0 1.5707 1.5707" xyz="0 0 0"/>
-      <inertia ixx="0.00052666666" ixy="0" ixz="0" iyy="0.00052666666" iyz="0" izz="0.001"/>
-    </inertial>
     <collision name="link_left_wheel_collision">
       <origin rpy="0 1.5707 1.5707" xyz="0 0 0" />
@@ -113,14 +109,11 @@
         <cylinder length="0.04" radius="0.1"/>
       </geometry>
+      <material name="orange"/>
     </visual>
+    <inertial>
+      <mass value="0.2"/>
+      <origin rpy="0 1.5707 1.5707" xyz="0 0 0"/>
+      <inertia ixx="0.00052666666" ixy="0" ixz="0" iyy="0.00052666666" iyz="0" izz="0.001"/>
+    </inertial>
   </link>
-  <!--   Joint for right wheel  -->
-  <joint name="joint_left_wheel" type="continuous">
-    <origin rpy="0 0 0" xyz="-0.05 -0.15 0"/>
-    <child link="link_left_wheel" />
-    <parent link="link_chassis"/>
-    <axis rpy="0 0 0" xyz="0 1 0"/>
-    <limit effort="10000" velocity="1000"/>
-    <joint_properties damping="1.0" friction="1.0" />
-  </joint>
 </robot>

Commit message: pu single logger into wall exit world

File: loggers_description/urdf/single_logger.urdf.xacro (robot description, xacro)
@@ -8,9 +8,9 @@
   <xacro:include filename="$(find loggers_description)/urdf/materials.xacro" />
   <!-- Used for fixing robot to Gazebo 'base_link' -->
-  <link name="world"/>
-  <joint name="joint_world_chassis" type="floating">
-    <parent link="world"/>
-    <child link="link_chassis"/>
-  </joint>
+  <!-- <link name="world"/> -->
+  <!-- <joint name="joint_world_chassis" type="planar"> -->
+  <!--   <parent link="world"/> -->
+  <!--   <child link="link_chassis"/> -->
+  <!-- </joint> -->
   <link name="link_chassis">
     <collision name="collision_chassis">
@@ -45,6 +45,6 @@
         <friction>
           <ode>
-            <mu>0</mu>
-            <mu2>0</mu2>
+            <mu>0.1</mu>
+            <mu2>0.1</mu2>
             <slip1>1.0</slip1>
             <slip2>1.0</slip2>

Commit message: add test script to single logger

File: loggers_description/urdf/single_logger.urdf.xacro (robot description, xacro)
@@ -27,7 +27,7 @@
     </visual>
     <inertial>
-      <mass value="5"/>
-      <origin rpy="0 0 0" xyz="0 0 0.1"/>
-      <inertia ixx="0.0395416666667" ixy="0" ixz="0" iyy="0.106208333333" iyz="0" izz="0.106208333333"/>
+      <mass value="2"/>
+      <origin rpy="0 0 0" xyz="0 0 0"/>
+      <inertia ixx="0.01582" ixy="0" ixz="0" iyy="0.04248" iyz="0" izz="0.05667"/>
     </inertial>
   </link>
@@ -38,5 +38,5 @@
   <link name="caster_front">
     <collision name="caster_front_collision">
-      <origin rpy=" 0 0 0" xyz="0.35 0 -0.05"/>
+      <origin rpy=" 0 0 0" xyz="0.2 0 -0.05"/>
       <geometry>
         <sphere radius="0.05"/>
@@ -45,6 +45,6 @@
         <friction>
           <ode>
-            <mu>0.1</mu>
-            <mu2>0.1</mu2>
+            <mu>0</mu>
+            <mu2>0</mu2>
             <slip1>1.0</slip1>
             <slip2>1.0</slip2>
@@ -60,4 +60,9 @@
       <material name="black"/>
     </visual>
+    <inertial>
+      <mass value="0.01"/>
+      <origin rpy="0 0 0" xyz="0 0 0"/>
+      <inertia ixx="0.001" ixy="0" ixz="0" iyy="0.001" iyz="0" izz="0.001"/>
+    </inertial>
   </link>
   <joint name="joint_right_wheel" type="continuous">
@@ -66,15 +71,15 @@
     <parent link="link_chassis"/>
     <axis rpy="0 0 0" xyz="0 1 0"/>
-    <limit effort="10000" velocity="1000"/>
-    <joint_properties damping="1.0" friction="1.0" />
+    <!-- <limit effort="10000" velocity="1000"/> -->
+    <!-- <joint_properties damping="1.0" friction="1.0" /> -->
   </joint>
   <link name="link_right_wheel">
     <inertial>
-      <mass value="0.2"/>
-      <origin rpy="0 1.5707 1.5707" xyz="0 0 0"/>
-      <inertia ixx="0.00052666666" ixy="0" ixz="0" iyy="0.00052666666" iyz="0" izz="0.001"/>
+      <mass value="0.01"/>
+      <origin rpy="0 0 0" xyz="0 0 0"/>
+      <inertia ixx="0.001" ixy="0" ixz="0" iyy="0.001" iyz="0" izz="0.001"/>
     </inertial>
     <collision name="link_right_wheel_collision">
-      <origin rpy="0 1.5707 1.5707" xyz="0 0 0" />
+      <origin rpy="0 ${PI/2} ${PI/2}" xyz="0 0 0" />
       <geometry>
         <cylinder length="0.04" radius="0.1"/>
@@ -82,5 +87,5 @@
     </collision>
     <visual name="link_right_wheel_visual">
-      <origin rpy="0 1.5707 1.5707" xyz="0 0 0"/>
+      <origin rpy="0 ${PI/2} ${PI/2}" xyz="0 0 0"/>
       <geometry>
         <cylinder length="0.04" radius="0.1"/>
@@ -94,10 +99,10 @@
     <parent link="link_chassis"/>
     <axis rpy="0 0 0" xyz="0 1 0"/>
-    <limit effort="10000" velocity="1000"/>
-    <joint_properties damping="1.0" friction="1.0" />
+    <!-- <limit effort="10000" velocity="1000"/> -->
+    <!-- <joint_properties damping="1.0" friction="1.0" /> -->
   </joint>
   <link name="link_left_wheel">
     <collision name="link_left_wheel_collision">
-      <origin rpy="0 1.5707 1.5707" xyz="0 0 0" />
+      <origin rpy="0 ${PI/2} ${PI/2}" xyz="0 0 0" />
       <geometry>
         <cylinder length="0.04" radius="0.1"/>
@@ -105,5 +110,5 @@
     </collision>
     <visual name="link_left_wheel_visual">
-      <origin rpy="0 1.5707 1.5707" xyz="0 0 0"/>
+      <origin rpy="0 ${PI/2} ${PI/2}" xyz="0 0 0"/>
       <geometry>
         <cylinder length="0.04" radius="0.1"/>
@@ -112,7 +117,7 @@
     </visual>
     <inertial>
-      <mass value="0.2"/>
-      <origin rpy="0 1.5707 1.5707" xyz="0 0 0"/>
-      <inertia ixx="0.00052666666" ixy="0" ixz="0" iyy="0.00052666666" iyz="0" izz="0.001"/>
+      <mass value="0.01"/>
+      <origin rpy="0 0 0" xyz="0 0 0"/>
+      <inertia ixx="0.001" ixy="0" ixz="0" iyy="0.001" iyz="0" izz="0.001"/>
     </inertial>
   </link>

Commit message: finish single logger world

File: loggers_description/urdf/single_logger.urdf.xacro (robot description, xacro)
@@ -7,10 +7,10 @@
   <!-- Import Rviz colors -->
   <xacro:include filename="$(find loggers_description)/urdf/materials.xacro" />
-  <!-- Used for fixing robot to Gazebo 'base_link' -->
-  <link name="world"/>
-  <joint name="joint_world_chassis" type="floating">
-    <parent link="world"/>
-    <child link="link_chassis"/>
-  </joint>
+  Used for fixing robot to Gazebo 'base_link'
+  <!-- <link name="world"/> -->
+  <!-- <joint name="joint_world_chassis" type="planar"> -->
+  <!--   <parent link="world"/> -->
+  <!--   <child link="link_chassis"/> -->
+  <!-- </joint> -->
   <link name="link_chassis">
     <visual>
@@ -54,7 +54,7 @@
     </collision>
     <inertial>
-      <mass value="0.01"/>
-      <origin rpy="0 0 0" xyz="0 0 0"/>
-      <inertia ixx="0.0001" ixy="0" ixz="0" iyy="0.0001" iyz="0" izz="0.0001"/>
+      <mass value="0.02"/>
+      <origin rpy="0 0 0" xyz="0 0 0"/>
+      <inertia ixx="0.00001" ixy="0" ixz="0" iyy="0.00001" iyz="0" izz="0.00001"/>
     </inertial>
   </link>
@@ -80,7 +80,7 @@
     </collision>
     <inertial>
-      <mass value="0.01"/>
-      <origin rpy="0 0 0" xyz="0 0 0"/>
-      <inertia ixx="0.0001" ixy="0" ixz="0" iyy="0.0001" iyz="0" izz="0.0001"/>
+      <mass value="0.02"/>
+      <origin rpy="0 0 0" xyz="0 0 0"/>
+      <inertia ixx="0.00001" ixy="0" ixz="0" iyy="0.00001" iyz="0" izz="0.00001"/>
     </inertial>
   </link>
@@ -106,5 +106,5 @@
     </collision>
     <inertial>
-      <mass value="0.02"/>
+      <mass value="0.04"/>
       <origin rpy="0 0 0" xyz="0 0 0"/>
       <inertia ixx="0.0001" ixy="0" ixz="0" iyy="0.0001" iyz="0" izz="0.0001"/>
@@ -190,3 +190,23 @@
     </inertial>
   </link>
+  <transmission name="trans_leftwheel">
+    <type>transmission_interface/SimpleTransmission</type>
+    <joint name="joint_chassis_leftwheel">
+      <hardwareInterface>hardware_interface/VelocityJointInterface</hardwareInterface>
+    </joint>
+    <actuator name="motor_leftwheel">
+      <hardwareInterface>hardware_interface/VelocityJointInterface</hardwareInterface>
+      <mechanicalReduction>1</mechanicalReduction>
+    </actuator>
+  </transmission>
+  <transmission name="trans_rightwheel">
+    <type>transmission_interface/SimpleTransmission</type>
+    <joint name="joint_chassis_rightwheel">
+      <hardwareInterface>hardware_interface/VelocityJointInterface</hardwareInterface>
+    </joint>
+    <actuator name="motor_rightwheel">
+      <hardwareInterface>hardware_interface/VelocityJointInterface</hardwareInterface>
+      <mechanicalReduction>1</mechanicalReduction>
+    </actuator>
+  </transmission>
 </robot>
