Commit message: change reward mechanism

File: loggers_description/urdf/single_logger.urdf.xacro (robot description, xacro)
@@ -8,107 +8,134 @@
   <xacro:include filename="$(find loggers_description)/urdf/materials.xacro" />
   Used for fixing robot to Gazebo 'base_link'
-  <!-- <link name="world"/> -->
-  <!-- <joint name="joint_world_chassis" type="planar"> -->
-  <!--   <parent link="world"/> -->
-  <!--   <child link="link_chassis"/> -->
+  <link name="world"/>
+  <joint name="joint_world_chassis" type="floating">
+    <parent link="world"/>
+    <child link="link_chassis"/>
+  </joint>
+  <link name="link_chassis">
+    <visual>
+      <origin rpy="0 0 0" xyz="0 0 0"/>
+      <geometry>
+        <box size="0.4 0.2 0.1"/>
+      </geometry>
+      <material name="uc_red"/>
+    </visual>
+    <collision>
+      <origin rpy="0 0 0" xyz="0 0 0"/>
+      <geometry>
+        <box size="0.4 0.2 0.1"/>
+      </geometry>
+    </collision>
+    <inertial>
+      <mass value="4"/>
+      <origin rpy="0 0 0" xyz="0 0 0"/>
+      <inertia ixx="0.01" ixy="0" ixz="0" iyy="0.01" iyz="0" izz="0.01"/>
+    </inertial>
+  </link>
+  <joint name="joint_chassis_caster" type="fixed">
+    <parent link="link_chassis"/>
+    <child link="link_caster"/>
+    <origin rpy="0 0 0" xyz="0.15 0 -0.05"/>
+  </joint>
+  <link name="link_caster">
+    <visual>
+      <origin rpy="0 0 0" xyz="0 0 0"/>
+      <geometry>
+        <sphere radius="0.04"/>
+      </geometry>
+      <material name="grey"/>
+    </visual>
+    <collision>
+      <origin rpy=" 0 0 0" xyz="0 0 0"/>
+      <geometry>
+        <sphere radius="0.04"/>
+      </geometry>
+    </collision>
+    <inertial>
+      <mass value="0.08"/>
+      <origin rpy="0 0 0" xyz="0 0 0"/>
+      <inertia ixx="0.0001" ixy="0" ixz="0" iyy="0.0001" iyz="0" izz="0.0001"/>
+    </inertial>
+  </link>
+  <!-- The following commented code experiment ball joint with 3 revolute joint, -->
+  <!-- however the behavior of the approximated ball joint was weird. -->
+  <!-- <joint name="joint_chassis_casterroll" type="continuous"> -->
+  <!--   <parent link="link_chassis"/> -->
+  <!--   <child link="link_caster_roll"/> -->
+  <!--   <origin rpy="0 0 0" xyz="0.15 0 -0.05"/> -->
+  <!--   <axis xyz="1 0 0"/> -->
   <!-- </joint> -->
-  <link name="link_chassis">
-    <visual>
-      <origin rpy="0 0 0" xyz="0 0 0"/>
-      <geometry>
-        <box size="0.4 0.2 0.1"/>
-      </geometry>
-      <material name="uc_red"/>
-    </visual>
-    <collision>
-      <origin rpy="0 0 0" xyz="0 0 0"/>
-      <geometry>
-        <box size="0.4 0.2 0.1"/>
-      </geometry>
-    </collision>
-    <inertial>
-      <mass value="2"/>
-      <origin rpy="0 0 0" xyz="0 0 0"/>
-      <inertia ixx="0.0083" ixy="0" ixz="0" iyy="0.0283" iyz="0" izz="0.0333"/>
-    </inertial>
-  </link>
-  <joint name="joint_chassis_casterroll" type="continuous">
-    <parent link="link_chassis"/>
-    <child link="link_caster_roll"/>
-    <origin rpy="0 0 0" xyz="0.15 0 -0.05"/>
-    <axis xyz="1 0 0"/>
-  </joint>
-  <link name="link_caster_roll">
-    <visual>
-      <origin rpy="0 0 0" xyz="0 0 0"/>
-      <geometry>
-        <sphere radius="0.00000001"/>
-      </geometry>
-      <material name="white"/>
-    </visual>
-    <collision>
-      <origin rpy=" 0 0 0" xyz="0 0 0"/>
-      <geometry>
-        <sphere radius="0.00000001"/>
-      </geometry>
-    </collision>
-    <inertial>
-      <mass value="0.02"/>
-      <origin rpy="0 0 0" xyz="0 0 0"/>
-      <inertia ixx="0.00001" ixy="0" ixz="0" iyy="0.00001" iyz="0" izz="0.00001"/>
-    </inertial>
-  </link>
-  <joint name="joint_casterroll_casterpitch" type="continuous">
-    <parent link="link_caster_roll"/>
-    <child link="link_caster_pitch"/>
-    <origin rpy="0 0 0" xyz="0 0 0"/>
-    <axis xyz="0 1 0"/>
-  </joint>
-  <link name="link_caster_pitch">
-    <visual>
-      <origin rpy="0 0 0" xyz="0 0 0"/>
-      <geometry>
-        <sphere radius="0.00000001"/>
-      </geometry>
-      <material name="white"/>
-    </visual>
-    <collision>
-      <origin rpy=" 0 0 0" xyz="0 0 0"/>
-      <geometry>
-        <sphere radius="0.00000001"/>
-      </geometry>
-    </collision>
-    <inertial>
-      <mass value="0.02"/>
-      <origin rpy="0 0 0" xyz="0 0 0"/>
-      <inertia ixx="0.00001" ixy="0" ixz="0" iyy="0.00001" iyz="0" izz="0.00001"/>
-    </inertial>
-  </link>
-  <joint name="joint_casterpitch_casteryaw" type="continuous">
-    <parent link="link_caster_pitch"/>
-    <child link="link_caster_yaw"/>
-    <origin rpy="0 0 0" xyz="0 0 0"/>
-    <axis xyz="0 0 1"/>
-  </joint>
-  <link name="link_caster_yaw">
-    <visual>
-      <origin rpy="0 0 0" xyz="0 0 0"/>
-      <geometry>
-        <sphere radius="0.04"/>
-      </geometry>
-      <material name="grey"/>
-    </visual>
-    <collision>
-      <origin rpy=" 0 0 0" xyz="0 0 0"/>
-      <geometry>
-        <sphere radius="0.04"/>
-      </geometry>
-    </collision>
-    <inertial>
-      <mass value="0.04"/>
-      <origin rpy="0 0 0" xyz="0 0 0"/>
-      <inertia ixx="0.0001" ixy="0" ixz="0" iyy="0.0001" iyz="0" izz="0.0001"/>
-    </inertial>
-  </link>
+  <!-- <link name="link_caster_roll"> -->
+  <!--   <visual> -->
+  <!--     <origin rpy="0 0 0" xyz="0 0 0"/> -->
+  <!--     <geometry> -->
+  <!--       <sphere radius="0.00000001"/> -->
+  <!--     </geometry> -->
+  <!--     <material name="white"/> -->
+  <!--   </visual> -->
+  <!--   <collision> -->
+  <!--     <origin rpy=" 0 0 0" xyz="0 0 0"/> -->
+  <!--     <geometry> -->
+  <!--       <sphere radius="0.00000001"/> -->
+  <!--     </geometry> -->
+  <!--   </collision> -->
+  <!--   <inertial> -->
+  <!--     <mass value="0.02"/> -->
+  <!--     <origin rpy="0 0 0" xyz="0 0 0"/> -->
+  <!--     <inertia ixx="0.00001" ixy="0" ixz="0" iyy="0.00001" iyz="0" izz="0.00001"/> -->
+  <!--   </inertial> -->
+  <!-- </link> -->
+  <!-- <joint name="joint_casterroll_casterpitch" type="continuous"> -->
+  <!--   <parent link="link_caster_roll"/> -->
+  <!--   <child link="link_caster_pitch"/> -->
+  <!--   <origin rpy="0 0 0" xyz="0 0 0"/> -->
+  <!--   <axis xyz="0 1 0"/> -->
+  <!-- </joint> -->
+  <!-- <link name="link_caster_pitch"> -->
+  <!--   <visual> -->
+  <!--     <origin rpy="0 0 0" xyz="0 0 0"/> -->
+  <!--     <geometry> -->
+  <!--       <sphere radius="0.00000001"/> -->
+  <!--     </geometry> -->
+  <!--     <material name="white"/> -->
+  <!--   </visual> -->
+  <!--   <collision> -->
+  <!--     <origin rpy=" 0 0 0" xyz="0 0 0"/> -->
+  <!--     <geometry> -->
+  <!--       <sphere radius="0.00000001"/> -->
+  <!--     </geometry> -->
+  <!--   </collision> -->
+  <!--   <inertial> -->
+  <!--     <mass value="0.02"/> -->
+  <!--     <origin rpy="0 0 0" xyz="0 0 0"/> -->
+  <!--     <inertia ixx="0.00001" ixy="0" ixz="0" iyy="0.00001" iyz="0" izz="0.00001"/> -->
+  <!--   </inertial> -->
+  <!-- </link> -->
+  <!-- <joint name="joint_casterpitch_casteryaw" type="continuous"> -->
+  <!--   <parent link="link_caster_pitch"/> -->
+  <!--   <child link="link_caster_yaw"/> -->
+  <!--   <origin rpy="0 0 0" xyz="0 0 0"/> -->
+  <!--   <axis xyz="0 0 1"/> -->
+  <!-- </joint> -->
+  <!-- <link name="link_caster_yaw"> -->
+  <!--   <visual> -->
+  <!--     <origin rpy="0 0 0" xyz="0 0 0"/> -->
+  <!--     <geometry> -->
+  <!--       <sphere radius="0.04"/> -->
+  <!--     </geometry> -->
+  <!--     <material name="grey"/> -->
+  <!--   </visual> -->
+  <!--   <collision> -->
+  <!--     <origin rpy=" 0 0 0" xyz="0 0 0"/> -->
+  <!--     <geometry> -->
+  <!--       <sphere radius="0.04"/> -->
+  <!--     </geometry> -->
+  <!--   </collision> -->
+  <!--   <inertial> -->
+  <!--     <mass value="0.04"/> -->
+  <!--     <origin rpy="0 0 0" xyz="0 0 0"/> -->
+  <!--     <inertia ixx="0.0001" ixy="0" ixz="0" iyy="0.0001" iyz="0" izz="0.0001"/> -->
+  <!--   </inertial> -->
+  <!-- </link> -->
   <joint name="joint_chassis_leftwheel" type="continuous">
     <origin rpy="0 0 0" xyz="-0.16 0.12 0.01"/>
@@ -132,5 +159,5 @@
     </collision>
     <inertial>
-      <mass value="0.02"/>
+      <mass value="0.2"/>
       <origin rpy="0 0 0" xyz="0 0 0"/>
       <inertia ixx="0.0001" ixy="0" ixz="0" iyy="0.0001" iyz="0" izz="0.0001"/>
@@ -158,7 +185,7 @@
     </visual>
     <inertial>
-      <mass value="0.01"/>
-      <origin rpy="0 0 0" xyz="0 0 0"/>
-      <inertia ixx="0.001" ixy="0" ixz="0" iyy="0.001" iyz="0" izz="0.001"/>
+      <mass value="02"/>
+      <origin rpy="0 0 0" xyz="0 0 0"/>
+      <inertia ixx="0.0001" ixy="0" ixz="0" iyy="0.0001" iyz="0" izz="0.0001"/>
     </inertial>
   </link>
@@ -185,7 +212,7 @@
     </collision>
     <inertial>
-      <mass value="0.01"/>
+      <mass value="0.1"/>
       <origin rpy="0 0 0" xyz="0 0 0.04"/>
-      <inertia ixx="0.00001" ixy="0" ixz="0" iyy="0.00001" iyz="0" izz="0.00001"/>
+      <inertia ixx="0.0001" ixy="0" ixz="0" iyy="0.0001" iyz="0" izz="0.0001"/>
     </inertial>
   </link>

Commit message: fix wheels weights, update diff_drive controller's config

File: loggers_description/urdf/single_logger.urdf.xacro (robot description, xacro)
@@ -185,5 +185,5 @@
     </visual>
     <inertial>
-      <mass value="02"/>
+      <mass value="0.2"/>
       <origin rpy="0 0 0" xyz="0 0 0"/>
       <inertia ixx="0.0001" ixy="0" ixz="0" iyy="0.0001" iyz="0" izz="0.0001"/>

Commit message: test two loggers, seems set model state may cause model crash

File: loggers_description/urdf/single_logger.urdf.xacro (robot description, xacro)
@@ -9,5 +9,5 @@
   <!-- Used for fixing robot to Gazebo 'base_link' -->
   <link name="world"/>
-  <joint name="joint_world_chassis" type="floating">
+  <joint name="joint_world_chassis" type="planar">
     <parent link="world"/>
     <child link="link_chassis"/>

File: loggers_description/urdf/two_loggers.urdf.xacro (robot description, xacro)
@@ -7,10 +7,10 @@
   <!-- Import Rviz colors -->
   <xacro:include filename="$(find loggers_description)/urdf/materials.xacro" />
-  <!-- Used for fixing robot to Gazebo 'base_link' -->
-  <!-- <link name="world"/> -->
-  <!-- <joint name="joint_world_chassis" type="planar"> -->
-  <!--   <parent link="world"/> -->
-  <!--   <child link="link_chassis"/> -->
-  <!-- </joint> -->
+  <!-- Use a dummy link, or Gazebo would not take care of root link's inertia -->
+  <link name="world"/>
+  <joint name="joint_world_chassis0" type="planar">
+    <parent link="world"/>
+    <child link="link_chassis_0"/>
+  </joint>
   <link name="link_chassis_0">
     <visual>

Commit message: use gazebo_ros_control plugin instead of ros-controllers plugin

File: loggers_description/urdf/single_logger.urdf.xacro (robot description, xacro)
@@ -9,5 +9,5 @@
   <!-- Used for fixing robot to Gazebo 'base_link' -->
   <link name="world"/>
-  <joint name="joint_world_chassis" type="planar">
+  <joint name="joint_world_chassis" type="floating">
     <parent link="world"/>
     <child link="link_chassis"/>

File: loggers_description/urdf/two_loggers.urdf.xacro (robot description, xacro)
@@ -11,6 +11,5 @@
   <!-- Use a dummy link, or Gazebo would not take care of root link's inertia -->
   <link name="world"/>
-  <joint name="joint_world_log" type="fixed">
-    <origin rpy="0 0 0" xyz="0 0 0"/>
+  <joint name="joint_world_log" type="floating">
     <parent link="world"/>
     <child link="link_log"/>
