Commit message: update two loggers urdf, set radius of chassis to 0.2

File: loggers_description/urdf/single_logger.urdf.xacro (robot description, xacro)
@@ -151,208 +151,4 @@
     </inertial>
   </link>
-  <!-- <link name="link_chassis"> -->
-  <!--   <visual> -->
-  <!--     <origin rpy="0 0 0" xyz="0 0 0"/> -->
-  <!--     <geometry> -->
-  <!--       <box size="0.4 0.2 0.1"/> -->
-  <!--     </geometry> -->
-  <!--     <material name="uc_red"/> -->
-  <!--   </visual> -->
-  <!--   <collision> -->
-  <!--     <origin rpy="0 0 0" xyz="0 0 0"/> -->
-  <!--     <geometry> -->
-  <!--       <box size="0.4 0.2 0.1"/> -->
-  <!--     </geometry> -->
-  <!--   </collision> -->
-  <!--   <inertial> -->
-  <!--     <mass value="4"/> -->
-  <!--     <origin rpy="0 0 0" xyz="0 0 0"/> -->
-  <!--     <inertia ixx="0.01" ixy="0" ixz="0" iyy="0.01" iyz="0" izz="0.01"/> -->
-  <!--   </inertial> -->
-  <!-- </link> -->
-  <!-- <joint name="joint_chassis_caster" type="fixed"> -->
-  <!--   <parent link="link_chassis"/> -->
-  <!--   <child link="link_caster"/> -->
-  <!--   <origin rpy="0 0 0" xyz="0.15 0 -0.05"/> -->
-  <!-- </joint>         -->
-  <!-- <link name="link_caster"> -->
-  <!--   <visual> -->
-  <!--     <origin rpy="0 0 0" xyz="0 0 0"/> -->
-  <!--     <geometry> -->
-  <!--       <sphere radius="0.04"/> -->
-  <!--     </geometry> -->
-  <!--     <material name="grey"/> -->
-  <!--   </visual> -->
-  <!--   <collision> -->
-  <!--     <origin rpy=" 0 0 0" xyz="0 0 0"/> -->
-  <!--     <geometry> -->
-  <!--       <sphere radius="0.04"/> -->
-  <!--     </geometry> -->
-  <!--   </collision> -->
-  <!--   <inertial> -->
-  <!--     <mass value="0.08"/> -->
-  <!--     <origin rpy="0 0 0" xyz="0 0 0"/> -->
-  <!--     <inertia ixx="0.0001" ixy="0" ixz="0" iyy="0.0001" iyz="0" izz="0.0001"/> -->
-  <!--   </inertial> -->
-  <!-- </link> -->
-  <!-- <!-\- The following commented code experiment ball joint with 3 revolute joint, -\-> -->
-  <!-- <!-\- however the behavior of the approximated ball joint was weird. -\-> -->
-  <!-- <!-\- <joint name="joint_chassis_casterroll" type="continuous"> -\-> -->
-  <!-- <!-\-   <parent link="link_chassis"/> -\-> -->
-  <!-- <!-\-   <child link="link_caster_roll"/> -\-> -->
-  <!-- <!-\-   <origin rpy="0 0 0" xyz="0.15 0 -0.05"/> -\-> -->
-  <!-- <!-\-   <axis xyz="1 0 0"/> -\-> -->
-  <!-- <!-\- </joint> -\->         -->
-  <!-- <!-\- <link name="link_caster_roll"> -\-> -->
-  <!-- <!-\-   <visual> -\-> -->
-  <!-- <!-\-     <origin rpy="0 0 0" xyz="0 0 0"/> -\-> -->
-  <!-- <!-\-     <geometry> -\-> -->
-  <!-- <!-\-       <sphere radius="0.00000001"/> -\-> -->
-  <!-- <!-\-     </geometry> -\-> -->
-  <!-- <!-\-     <material name="white"/> -\-> -->
-  <!-- <!-\-   </visual> -\-> -->
-  <!-- <!-\-   <collision> -\-> -->
-  <!-- <!-\-     <origin rpy=" 0 0 0" xyz="0 0 0"/> -\-> -->
-  <!-- <!-\-     <geometry> -\-> -->
-  <!-- <!-\-       <sphere radius="0.00000001"/> -\-> -->
-  <!-- <!-\-     </geometry> -\-> -->
-  <!-- <!-\-   </collision> -\-> -->
-  <!-- <!-\-   <inertial> -\-> -->
-  <!-- <!-\-     <mass value="0.02"/> -\-> -->
-  <!-- <!-\-     <origin rpy="0 0 0" xyz="0 0 0"/> -\-> -->
-  <!-- <!-\-     <inertia ixx="0.00001" ixy="0" ixz="0" iyy="0.00001" iyz="0" izz="0.00001"/> -\-> -->
-  <!-- <!-\-   </inertial> -\-> -->
-  <!-- <!-\- </link> -\-> -->
-  <!-- <!-\- <joint name="joint_casterroll_casterpitch" type="continuous"> -\-> -->
-  <!-- <!-\-   <parent link="link_caster_roll"/> -\-> -->
-  <!-- <!-\-   <child link="link_caster_pitch"/> -\-> -->
-  <!-- <!-\-   <origin rpy="0 0 0" xyz="0 0 0"/> -\-> -->
-  <!-- <!-\-   <axis xyz="0 1 0"/> -\-> -->
-  <!-- <!-\- </joint> -\-> -->
-  <!-- <!-\- <link name="link_caster_pitch"> -\-> -->
-  <!-- <!-\-   <visual> -\-> -->
-  <!-- <!-\-     <origin rpy="0 0 0" xyz="0 0 0"/> -\-> -->
-  <!-- <!-\-     <geometry> -\-> -->
-  <!-- <!-\-       <sphere radius="0.00000001"/> -\-> -->
-  <!-- <!-\-     </geometry> -\-> -->
-  <!-- <!-\-     <material name="white"/> -\-> -->
-  <!-- <!-\-   </visual> -\-> -->
-  <!-- <!-\-   <collision> -\-> -->
-  <!-- <!-\-     <origin rpy=" 0 0 0" xyz="0 0 0"/> -\-> -->
-  <!-- <!-\-     <geometry> -\-> -->
-  <!-- <!-\-       <sphere radius="0.00000001"/> -\-> -->
-  <!-- <!-\-     </geometry> -\-> -->
-  <!-- <!-\-   </collision> -\-> -->
-  <!-- <!-\-   <inertial> -\-> -->
-  <!-- <!-\-     <mass value="0.02"/> -\-> -->
-  <!-- <!-\-     <origin rpy="0 0 0" xyz="0 0 0"/> -\-> -->
-  <!-- <!-\-     <inertia ixx="0.00001" ixy="0" ixz="0" iyy="0.00001" iyz="0" izz="0.00001"/> -\-> -->
-  <!-- <!-\-   </inertial> -\-> -->
-  <!-- <!-\- </link> -\-> -->
-  <!-- <!-\- <joint name="joint_casterpitch_casteryaw" type="continuous"> -\-> -->
-  <!-- <!-\-   <parent link="link_caster_pitch"/> -\-> -->
-  <!-- <!-\-   <child link="link_caster_yaw"/> -\-> -->
-  <!-- <!-\-   <origin rpy="0 0 0" xyz="0 0 0"/> -\-> -->
-  <!-- <!-\-   <axis xyz="0 0 1"/> -\-> -->
-  <!-- <!-\- </joint> -\-> -->
-  <!-- <!-\- <link name="link_caster_yaw"> -\-> -->
-  <!-- <!-\-   <visual> -\-> -->
-  <!-- <!-\-     <origin rpy="0 0 0" xyz="0 0 0"/> -\-> -->
-  <!-- <!-\-     <geometry> -\-> -->
-  <!-- <!-\-       <sphere radius="0.04"/> -\-> -->
-  <!-- <!-\-     </geometry> -\-> -->
-  <!-- <!-\-     <material name="grey"/> -\-> -->
-  <!-- <!-\-   </visual> -\-> -->
-  <!-- <!-\-   <collision> -\-> -->
-  <!-- <!-\-     <origin rpy=" 0 0 0" xyz="0 0 0"/> -\-> -->
-  <!-- <!-\-     <geometry> -\-> -->
-  <!-- <!-\-       <sphere radius="0.04"/> -\-> -->
-  <!-- <!-\-     </geometry> -\-> -->
-  <!-- <!-\-   </collision> -\-> -->
-  <!-- <!-\-   <inertial> -\-> -->
-  <!-- <!-\-     <mass value="0.04"/> -\-> -->
-  <!-- <!-\-     <origin rpy="0 0 0" xyz="0 0 0"/> -\-> -->
-  <!-- <!-\-     <inertia ixx="0.0001" ixy="0" ixz="0" iyy="0.0001" iyz="0" izz="0.0001"/> -\-> -->
-  <!-- <!-\-   </inertial> -\-> -->
-  <!-- <!-\- </link> -\-> -->
-  <!-- <joint name="joint_chassis_leftwheel" type="continuous"> -->
-  <!--   <origin rpy="0 0 0" xyz="-0.16 0.12 0.01"/> -->
-  <!--   <child link="link_left_wheel" /> -->
-  <!--   <parent link="link_chassis"/> -->
-  <!--   <axis rpy="0 0 0" xyz="0 1 0"/> -->
-  <!-- </joint>   -->
-  <!-- <link name="link_left_wheel">     -->
-  <!--   <visual> -->
-  <!--     <origin rpy="${PI/2} 0 0" xyz="0 0 0"/> -->
-  <!--     <geometry> -->
-  <!--       <cylinder length="0.04" radius="0.1"/> -->
-  <!--     </geometry> -->
-  <!--     <material name="black"/> -->
-  <!--   </visual> -->
-  <!--   <collision> -->
-  <!--     <origin rpy="${PI/2} 0 0" xyz="0 0 0" /> -->
-  <!--     <geometry> -->
-  <!--       <cylinder length="0.04" radius="0.1"/> -->
-  <!--     </geometry> -->
-  <!--   </collision> -->
-  <!--   <inertial> -->
-  <!--     <mass value="0.2"/> -->
-  <!--     <origin rpy="0 0 0" xyz="0 0 0"/> -->
-  <!--     <inertia ixx="0.0001" ixy="0" ixz="0" iyy="0.0001" iyz="0" izz="0.0001"/> -->
-  <!--   </inertial> -->
-  <!-- </link> -->
-  <!-- <joint name="joint_chassis_rightwheel" type="continuous"> -->
-  <!--   <origin rpy="0 0 0" xyz="-0.16 -0.12 0.01"/> -->
-  <!--   <child link="link_right_wheel" /> -->
-  <!--   <parent link="link_chassis"/> -->
-  <!--   <axis rpy="0 0 0" xyz="0 1 0"/> -->
-  <!-- </joint>     -->
-  <!-- <link name="link_right_wheel">     -->
-  <!--   <collision> -->
-  <!--     <origin rpy="${PI/2} 0 0" xyz="0 0 0" /> -->
-  <!--     <geometry> -->
-  <!--       <cylinder length="0.04" radius="0.1"/> -->
-  <!--     </geometry> -->
-  <!--   </collision> -->
-  <!--   <visual> -->
-  <!--     <origin rpy="${PI/2} 0 0" xyz="0 0 0"/> -->
-  <!--     <geometry> -->
-  <!--       <cylinder length="0.04" radius="0.1"/> -->
-  <!--     </geometry> -->
-  <!--     <material name="black"/> -->
-  <!--   </visual> -->
-  <!--   <inertial> -->
-  <!--     <mass value="0.2"/> -->
-  <!--     <origin rpy="0 0 0" xyz="0 0 0"/> -->
-  <!--     <inertia ixx="0.0001" ixy="0" ixz="0" iyy="0.0001" iyz="0" izz="0.0001"/> -->
-  <!--   </inertial> -->
-  <!-- </link> -->
-  <!-- <joint name="joint_chassis_hat" type="revolute"> -->
-  <!--   <origin rpy="0 0 0" xyz="0.0 0 0.05"/> -->
-  <!--   <limit effort="0" lower="0" upper="0" velocity="0"/> -->
-  <!--   <child link="link_hat" /> -->
-  <!--   <parent link="link_chassis"/> -->
-  <!--   <axis rpy="0 0 0" xyz="0 0 1"/> -->
-  <!-- </joint>     -->
-  <!-- <link name="link_hat"> -->
-  <!--   <visual> -->
-  <!--     <origin rpy="0 0 0" xyz="0 0 0.04"/> -->
-  <!--     <geometry> -->
-  <!--       <cylinder length="0.08" radius="0.02"/> -->
-  <!--     </geometry> -->
-  <!--     <material name="uc_red"/> -->
-  <!--   </visual> -->
-  <!--   <collision> -->
-  <!--     <origin rpy="0 0 0" xyz="0 0 0.04"/> -->
-  <!--     <geometry> -->
-  <!--       <cylinder length="0.08" radius="0.02"/> -->
-  <!--     </geometry> -->
-  <!--   </collision> -->
-  <!--   <inertial> -->
-  <!--     <mass value="0.1"/> -->
-  <!--     <origin rpy="0 0 0" xyz="0 0 0.04"/> -->
-  <!--     <inertia ixx="0.0001" ixy="0" ixz="0" iyy="0.0001" iyz="0" izz="0.0001"/> -->
-  <!--   </inertial> -->
-  <!-- </link> -->
   <!-- <transmission name="trans_leftwheel"> -->
   <!--   <type>transmission_interface/SimpleTransmission</type> -->

File: loggers_description/urdf/two_loggers.urdf.xacro (robot description, xacro)
@@ -13,5 +13,5 @@
   <xacro:property name="M_HAT" value="0.5"/>
   <!-- properties of link_chassis* -->
-  <xacro:property name="R_CHASSIS" value="0.4"/>
+  <xacro:property name="R_CHASSIS" value="0.2"/>
   <xacro:property name="L_CHASSIS" value="0.1"/>
   <xacro:property name="M_CHASSIS" value="2"/>

Commit message: upgrade solo env to adpative dynamic world

File: loggers_description/urdf/single_logger.urdf.xacro (robot description, xacro)
@@ -8,5 +8,5 @@
   <xacro:property name="M_HAT" value="0.5"/>
   <!-- properties of link_chassis -->
-  <xacro:property name="R_CHASSIS" value="0.2"/>
+  <xacro:property name="R_CHASSIS" value="0.25"/>
   <xacro:property name="L_CHASSIS" value="0.1"/>
   <xacro:property name="M_CHASSIS" value="2"/>
