Commit message: update solo logger related files

File: loggers_description/urdf/logger.urdf.xacro (robot description, xacro)
@@ -23,5 +23,5 @@
     <xacro:include filename="$(find loggers_description)/urdf/materials.xacro" />
     <!-- building the robot in following-->
-    <xacro:macro name="logger_base_macro">
+    <xacro:macro name="logger_macro">
         <link name="chassis">
             <visual>
@@ -118,5 +118,5 @@
             <material>Gazebo/Wood</material>
         </gazebo>
-        <joint name="chassis_right_wheel" type="continuous">
+        <joint name="chassis-right_wheel" type="continuous">
             <origin rpy="0 0 0" xyz="${-R_CHASSIS/2} ${R_CHASSIS/2} 0"/>
             <child link="right_wheel" />
@@ -181,4 +181,22 @@
         <material>Gazebo/Red</material>
     </gazebo>
+    <!-- differential_drive_controller plugin -->
+    <gazebo>
+        <plugin name="differential_drive_controller" filename="libgazebo_ros_diff_drive.so">
+            <legacyMode>false</legacyMode>
+            <alwaysOn>true</alwaysOn>
+            <updateRate>100</updateRate>
+            <leftJoint>chassis-left_wheel</leftJoint>
+            <rightJoint>chassis-right_wheel</rightJoint>
+            <wheelSeparation>0.25</wheelSeparation>
+            <wheelDiameter>0.18</wheelDiameter>
+            <wheelTorque>1</wheelTorque>
+            <!--wheelAcceleration>${wheel_accel}</wheelAcceleration-->
+            <commandTopic>cmd_vel_0</commandTopic>
+            <odometryTopic>odom</odometryTopic>
+            <odometryFrame>odom</odometryFrame>
+            <robotBaseFrame>chassis</robotBaseFrame>
+        </plugin>
+    </gazebo>
     </xacro:macro>
 </robot>

File: loggers_description/urdf/logger_0.urdf.xacro (robot description, xacro)
@@ -4,4 +4,4 @@
     <xacro:include filename="$(find loggers_description)/urdf/logger.urdf.xacro" />
     <!-- Instantiate logger_base_macro once (has no parameters atm) -->
-    <xacro:logger_base_macro />
+    <xacro:logger_macro />
 </robot>

Commit message: update logger urdf so that logger forward align with +x

File: loggers_description/urdf/logger.urdf.xacro (robot description, xacro)
@@ -23,6 +23,6 @@
     <xacro:include filename="$(find loggers_description)/urdf/materials.xacro" />
     <!-- building the robot in following-->
-    <xacro:macro name="logger_macro">
-        <link name="chassis">
+    <xacro:macro name="logger_macro" params="model_name">
+        <link name="${model_name}-chassis">
             <visual>
                 <origin rpy="0 0 0" xyz="0 0 0"/>
@@ -39,5 +39,5 @@
             </collision>
         </link>
-        <gazebo reference="chassis">
+        <gazebo reference="${model_name}-chassis">
             <mu1>0.2</mu1>
             <mu2>0.2</mu2>
@@ -45,10 +45,10 @@
         </gazebo>
         <!-- kdl does not support a root link with an inertia, create a dummy link only contains inertia of base_link -->
-        <joint name="chassis-cha_inertial" type="fixed">
+        <joint name="${model_name}-chassis2cha_inertial" type="fixed">
             <origin xyz="0 0 0" rpy="0 0 0" />
-            <parent link="chassis" />
-            <child link="cha_inertial" />
-        </joint>
-        <link name="cha_inertial">
+            <parent link="${model_name}-chassis" />
+            <child link="${model_name}-cha_inertial" />
+        </joint>
+        <link name="${model_name}-cha_inertial">
             <inertial>
                 <mass value="${M_CHASSIS}"/>
@@ -57,10 +57,10 @@
             </inertial>
         </link>
-        <joint name="chassis-caster" type="fixed">
-            <origin rpy="0 0 0" xyz="0 ${-R_CHASSIS/2} ${-L_CHASSIS/2}"/>
-            <parent link="chassis"/>
-            <child link="caster"/>
-        </joint>
-        <link name="caster">
+        <joint name="${model_name}-chassis2caster" type="fixed">
+            <origin rpy="0 0 0" xyz="${R_CHASSIS/2} 0 ${-L_CHASSIS/2}"/>
+            <parent link="${model_name}-chassis"/>
+            <child link="${model_name}-caster"/>
+        </joint>
+        <link name="${model_name}-caster">
             <visual>
                 <origin rpy="0 0 0" xyz="0 0 0"/>
@@ -82,18 +82,18 @@
             </inertial>
         </link>
-        <gazebo reference="caster">
+        <gazebo reference="${model_name}-caster">
             <mu1>0.0</mu1>
             <mu2>0.0</mu2>
             <material>Gazebo/Grey</material>
         </gazebo>
-        <joint name="chassis-left_wheel" type="continuous">
-            <origin rpy="0 0 0" xyz="${R_CHASSIS/2} ${R_CHASSIS/2} 0"/>
-            <parent link="chassis"/>
-            <child link="left_wheel" />
-            <axis rpy="0 0 0" xyz="1 0 0"/>
-        </joint>
-        <link name="left_wheel">
-            <visual>
-                <origin rpy="0 ${PI/2} 0" xyz="0 0 0"/>
+        <joint name="${model_name}-chassis2left_wheel" type="continuous">
+            <origin rpy="0 0 0" xyz="${-R_CHASSIS/2} ${-R_CHASSIS/2} 0"/>
+            <parent link="${model_name}-chassis"/>
+            <child link="${model_name}-left_wheel" />
+            <axis rpy="0 0 0" xyz="0 1 0"/>
+        </joint>
+        <link name="${model_name}-left_wheel">
+            <visual>
+                <origin rpy="${PI/2} 0 0" xyz="0 0 0"/>
                 <geometry>
                     <cylinder length="${L_WHEEL}" radius="${R_WHEEL}"/>
@@ -102,5 +102,5 @@
             </visual>
             <collision>
-                <origin rpy="0 ${PI/2} 0" xyz="0 0 0" />
+                <origin rpy="${PI/2} 0 0" xyz="0 0 0" />
                 <geometry>
                     <cylinder length="${L_WHEEL}" radius="${R_WHEEL}"/>
@@ -109,28 +109,28 @@
             <inertial>
                 <mass value="${M_WHEEL}"/>
-                <origin rpy="0 ${PI/2} 0" xyz="0 0 0"/>
+                <origin rpy="${PI/2} 0 0" xyz="0 0 0"/>
                 <inertia ixx="${1/12*M_WHEEL*(3*R_WHEEL*R_WHEEL+L_WHEEL*L_WHEEL)}" ixy="0" ixz="0" iyy="${1/12*M_WHEEL*(3*R_WHEEL*R_WHEEL+L_WHEEL*L_WHEEL)}" iyz="0" izz="${1/2*M_WHEEL*R_WHEEL*R_WHEEL}"/>
             </inertial>
         </link>
-        <gazebo reference="left_wheel">
+        <gazebo reference="${model_name}-left_wheel">
             <mu1>0.99</mu1>
             <mu2>0.99</mu2>
             <material>Gazebo/Wood</material>
         </gazebo>
-        <joint name="chassis-right_wheel" type="continuous">
+        <joint name="${model_name}-chassis2right_wheel" type="continuous">
             <origin rpy="0 0 0" xyz="${-R_CHASSIS/2} ${R_CHASSIS/2} 0"/>
-            <child link="right_wheel" />
-            <parent link="chassis"/>
-            <axis rpy="0 0 0" xyz="1 0 0"/>
-        </joint>
-        <link name="right_wheel">
-            <collision>
-                <origin rpy="0 ${PI/2} 0" xyz="0 0 0" />
-                <geometry>
-                    <cylinder length="${L_WHEEL}" radius="${R_WHEEL}"/>
-                </geometry>
-            </collision>
-            <visual>
-                <origin rpy="0 ${PI/2} 0" xyz="0 0 0"/>
+            <parent link="${model_name}-chassis"/>
+            <child link="${model_name}-right_wheel" />
+            <axis rpy="0 0 0" xyz="0 1 0"/>
+        </joint>
+        <link name="${model_name}-right_wheel">
+            <collision>
+                <origin rpy="${PI/2} 0 0" xyz="0 0 0" />
+                <geometry>
+                    <cylinder length="${L_WHEEL}" radius="${R_WHEEL}"/>
+                </geometry>
+            </collision>
+            <visual>
+                <origin rpy="${PI/2} 0 0" xyz="0 0 0"/>
                 <geometry>
                     <cylinder length="${L_WHEEL}" radius="${R_WHEEL}"/>
@@ -140,21 +140,20 @@
             <inertial>
                 <mass value="${M_WHEEL}"/>
-                <origin rpy="0 ${PI/2} 0" xyz="0 0 0"/>
+                <origin rpy="${PI/2} 0 0" xyz="0 0 0"/>
                 <inertia ixx="${1/12*M_WHEEL*(3*R_WHEEL*R_WHEEL+L_WHEEL*L_WHEEL)}" ixy="0" ixz="0" iyy="${1/12*M_WHEEL*(3*R_WHEEL*R_WHEEL+L_WHEEL*L_WHEEL)}" iyz="0" izz="${1/2*M_WHEEL*R_WHEEL*R_WHEEL}"/>
             </inertial>
         </link>
-        <gazebo reference="right_wheel">
+        <gazebo reference="${model_name}-right_wheel">
             <mu1>0.99</mu1>
             <mu2>0.99</mu2>
             <material>Gazebo/Wood</material>
         </gazebo>
-    <joint name="joint_chassis_hat" type="continuous">
+    <joint name="${model_name}-chassis2hat" type="continuous">
         <origin rpy="0 0 0" xyz="0.0 0 ${(L_HAT+L_CHASSIS)/2}"/>
-        <limit effort="0" lower="0" upper="0" velocity="0"/>
-        <parent link="chassis"/>
-        <child link="hat" />
+        <parent link="${model_name}-chassis"/>
+        <child link="${model_name}-hat" />
         <axis rpy="0 0 0" xyz="0 0 1"/>
     </joint>
-    <link name="hat">
+    <link name="${model_name}-hat">
         <visual>
             <origin rpy="0 0 0" xyz="0 0 0"/>
@@ -176,5 +175,5 @@
         </inertial>
     </link>
-    <gazebo reference="hat">
+    <gazebo reference="${model_name}-hat">
         <mu1>0</mu1>
         <mu2>0</mu2>

File: loggers_description/urdf/solo_logger.urdf.xacro (robot description, xacro)
@@ -4,5 +4,5 @@
     <xacro:include filename="$(find loggers_description)/urdf/logger.urdf.xacro" />
     <!-- Instantiate logger_base_macro once (has no parameters atm) -->
-    <xacro:logger_macro />
+    <xacro:logger_macro model_name="logger"/>
     <!-- differential_drive_controller plugin -->
     <gazebo>
@@ -11,6 +11,6 @@
             <alwaysOn>true</alwaysOn>
             <updateRate>100</updateRate>
-            <leftJoint>chassis-left_wheel</leftJoint>
-            <rightJoint>chassis-right_wheel</rightJoint>
+            <leftJoint>logger-chassis2left_wheel</leftJoint>
+            <rightJoint>logger-chassis2right_wheel</rightJoint>
             <wheelSeparation>0.25</wheelSeparation>
             <wheelDiameter>0.18</wheelDiameter>
@@ -19,5 +19,5 @@
             <odometryTopic>odom</odometryTopic>
             <odometryFrame>odom</odometryFrame>
-            <robotBaseFrame>chassis</robotBaseFrame>
+            <robotBaseFrame>logger-chassis</robotBaseFrame>
         </plugin>
     </gazebo>
