Commit message: add more gazebo properties to links in urdf, hoping to supress model blown

File: loggers_description/urdf/double_logger_2wd.urdf.xacro (robot description, xacro)
@@ -7,5 +7,5 @@
     <!-- Included URDF Files -->
     <xacro:include filename="$(find loggers_description)/urdf/logger.urdf.xacro" />
-    <xacro:include filename="$(find loggers_description)/urdf/logger_copy.urdf.xacro" />
+    <xacro:include filename="$(find loggers_description)/urdf/logger_copy_fixedhat.urdf.xacro" />
     <!-- Instantiate logger_base_macro once (has no parameters atm) -->
     <xacro:logger_macro model_name="logger0"/>
@@ -55,11 +55,7 @@
     </link>
     <gazebo reference="log">
+        <mu1>0</mu1>
+        <mu2>0</mu2>
         <material>Gazebo/Wood</material>
-        <dampingFactor>0.02</dampingFactor>
-        <maxVel>0.1</maxVel>
-        <minDepth>0.01</minDepth>
-        <selfCollide>true</selfCollide>
-        <mu1>0.99</mu1>
-        <mu2>0.99</mu2>
     </gazebo>
     <!-- Instantiate logger_base_macro once (has no parameters atm) -->

File: loggers_description/urdf/logger_copy.urdf.xacro (robot description, xacro)
@@ -50,7 +50,11 @@
         </link>
         <gazebo reference="${model_name}-hat">
-            <mu1>0</mu1>
-            <mu2>0</mu2>
             <material>Gazebo/Red</material>
+            <dampingFactor>0.02</dampingFactor>
+            <maxVel>0.1</maxVel>
+            <minDepth>0.01</minDepth>
+            <selfCollide>true</selfCollide>
+            <mu1>0.99</mu1>
+            <mu2>0.99</mu2>
         </gazebo>
         <joint name="${model_name}-hat2chassis" type="continuous">
@@ -81,7 +85,11 @@
         </link>
         <gazebo reference="${model_name}-chassis">
-            <mu1>0.5</mu1>
-            <mu2>0.5</mu2>
             <material>Gazebo/Black</material>
+            <dampingFactor>0.02</dampingFactor>
+            <maxVel>0.1</maxVel>
+            <minDepth>0.01</minDepth>
+            <selfCollide>true</selfCollide>
+            <mu1>0.99</mu1>
+            <mu2>0.99</mu2>
         </gazebo>
         <joint name="${model_name}-chassis2caster" type="fixed">
@@ -111,7 +119,11 @@
         </link>
         <gazebo reference="${model_name}-caster">
+            <material>Gazebo/Grey</material>
+            <dampingFactor>0.02</dampingFactor>
+            <maxVel>0.1</maxVel>
+            <minDepth>0.01</minDepth>
+            <selfCollide>true</selfCollide>
             <mu1>0.0</mu1>
             <mu2>0.0</mu2>
-            <material>Gazebo/Grey</material>
         </gazebo>
         <joint name="${model_name}-chassis2left_wheel" type="continuous">
@@ -142,7 +154,11 @@
         </link>
         <gazebo reference="${model_name}-left_wheel">
-            <mu1>0.99</mu1>
-            <mu2>0.99</mu2>
             <material>Gazebo/Wood</material>
+            <dampingFactor>0.02</dampingFactor>
+            <maxVel>100</maxVel>
+            <minDepth>0.01</minDepth>
+            <selfCollide>true</selfCollide>
+            <mu1>0.99</mu1>
+            <mu2>0.99</mu2>
         </gazebo>
         <joint name="${model_name}-chassis2right_wheel" type="continuous">
@@ -173,7 +189,11 @@
         </link>
         <gazebo reference="${model_name}-right_wheel">
-            <mu1>0.99</mu1>
-            <mu2>0.99</mu2>
             <material>Gazebo/Wood</material>
+            <dampingFactor>0.02</dampingFactor>
+            <maxVel>100</maxVel>
+            <minDepth>0.01</minDepth>
+            <selfCollide>true</selfCollide>
+            <mu1>0.99</mu1>
+            <mu2>0.99</mu2>
         </gazebo>
     </xacro:macro>

File: loggers_description/urdf/logger_copy_fixedhat.urdf.xacro (robot description, xacro)
@@ -18,10 +18,47 @@
     <xacro:property name="L_WHEEL" value="0.04"/>
     <xacro:property name="M_WHEEL" value="0.5"/>
-    <!-- Import all Gazebo-customization elements, including Gazebo colors -->
-    <!-- <xacro:include filename="$(find loggers_description)/urdf/single_logger.gazebo" /> -->
     <!-- Import Rviz colors -->
-    <xacro:include filename="$(find loggers_description)/urdf/materials.xacro" />
+    <!-- <xacro:include filename="$(find loggers_description)/urdf/materials.xacro" /> -->
     <!-- building the robot in following-->
-    <xacro:macro name="logger_macro" params="model_name">
+    <xacro:macro name="logger_copy_macro" params="model_name parent *origin">
+        <joint name="${parent}2${model_name}-hat" type="revolute">
+            <xacro:insert_block name="origin" />
+            <parent link="${parent}"/>
+            <child link="${model_name}-hat"/>
+            <limit lower="0" upper="0" effort="0" velocity="0"/>
+            <axis xyz="0 0 1"/>
+        </joint>
+        <link name="${model_name}-hat">
+            <visual>
+                <origin rpy="0 0 0" xyz="0 0 ${-L_HAT/2}"/>
+                <geometry>
+                    <cylinder length="${L_HAT}" radius="${R_HAT}"/>
+                </geometry>
+                <material name="red"/>
+            </visual>
+            <collision>
+                <origin rpy="0 0 0" xyz="0 0 ${-L_HAT/2}"/>
+                <geometry>
+                    <cylinder length="${L_HAT}" radius="${R_HAT}"/>
+                </geometry>
+            </collision>
+            <inertial>
+                <mass value="${M_HAT}"/>
+                <origin rpy="0 0 0" xyz="0 0 ${-L_HAT/2}"/>
+                <inertia ixx="${1/12*M_HAT*(3*R_HAT*R_HAT+L_HAT*L_HAT)}" ixy="0" ixz="0" iyy="${1/12*M_HAT*(3*R_HAT*R_HAT+L_HAT*L_HAT)}" iyz="0" izz="${1/2*M_HAT*R_HAT*R_HAT}"/>
+            </inertial>
+        </link>
+        <gazebo reference="${model_name}-hat">
+            <mu1>0</mu1>
+            <mu2>0</mu2>
+            <material>Gazebo/Red</material>
+        </gazebo>
+        <joint name="${model_name}-hat2chassis" type="revolute">
+            <origin rpy="0 0 ${PI/2}" xyz="0.0 0 ${-L_HAT+-L_CHASSIS/2}"/>
+            <parent link="${model_name}-hat" />
+            <child link="${model_name}-chassis"/>
+            <limit effort="0" lower="0" upper="0" velocity="0"/>
+            <axis rpy="0 0 0" xyz="0 0 1"/>
+        </joint>
         <link name="${model_name}-chassis">
             <visual>
@@ -30,5 +67,5 @@
                     <cylinder length="${L_CHASSIS}" radius="${R_CHASSIS}"/>
                 </geometry>
-                <material name="white"/>
+                <material name="black"/>
             </visual>
             <collision>
@@ -38,21 +75,4 @@
                 </geometry>
             </collision>
-        </link>
-        <gazebo reference="${model_name}-chassis">
-            <material>Gazebo/White</material>
-            <dampingFactor>0.02</dampingFactor>
-            <maxVel>0.1</maxVel>
-            <minDepth>0.01</minDepth>
-            <selfCollide>true</selfCollide>
-            <mu1>0.99</mu1>
-            <mu2>0.99</mu2>
-        </gazebo>
-        <!-- kdl does not support a root link with an inertia, create a dummy link only contains inertia of base_link -->
-        <joint name="${model_name}-chassis2cha_inertial" type="fixed">
-            <origin xyz="0 0 0" rpy="0 0 0" />
-            <parent link="${model_name}-chassis" />
-            <child link="${model_name}-cha_inertial" />
-        </joint>
-        <link name="${model_name}-cha_inertial">
             <inertial>
                 <mass value="${M_CHASSIS}"/>
@@ -61,4 +81,9 @@
             </inertial>
         </link>
+        <gazebo reference="${model_name}-chassis">
+            <mu1>0.5</mu1>
+            <mu2>0.5</mu2>
+            <material>Gazebo/Black</material>
+        </gazebo>
         <joint name="${model_name}-chassis2caster" type="fixed">
             <origin rpy="0 0 0" xyz="${R_CHASSIS/2} 0 ${-L_CHASSIS/2}"/>
@@ -87,11 +112,7 @@
         </link>
         <gazebo reference="${model_name}-caster">
-            <material>Gazebo/Grey</material>
-            <dampingFactor>0.02</dampingFactor>
-            <maxVel>0.1</maxVel>
-            <minDepth>0.01</minDepth>
-            <selfCollide>true</selfCollide>
             <mu1>0.0</mu1>
             <mu2>0.0</mu2>
+            <material>Gazebo/Grey</material>
         </gazebo>
         <joint name="${model_name}-chassis2left_wheel" type="continuous">
@@ -122,11 +143,7 @@
         </link>
         <gazebo reference="${model_name}-left_wheel">
-            <material>Gazebo/Wood</material>
-            <dampingFactor>0.02</dampingFactor>
-            <maxVel>100</maxVel>
-            <minDepth>0.01</minDepth>
-            <selfCollide>true</selfCollide>
             <mu1>0.99</mu1>
             <mu2>0.99</mu2>
+            <material>Gazebo/Wood</material>
         </gazebo>
         <joint name="${model_name}-chassis2right_wheel" type="continuous">
@@ -157,46 +174,7 @@
         </link>
         <gazebo reference="${model_name}-right_wheel">
-            <material>Gazebo/Wood</material>
-            <dampingFactor>0.02</dampingFactor>
-            <maxVel>100</maxVel>
-            <minDepth>0.01</minDepth>
-            <selfCollide>true</selfCollide>
             <mu1>0.99</mu1>
             <mu2>0.99</mu2>
-        </gazebo>
-        <joint name="${model_name}-chassis2hat" type="continuous">
-            <origin rpy="0 0 0" xyz="0.0 0 ${(L_HAT+L_CHASSIS)/2}"/>
-            <parent link="${model_name}-chassis"/>
-            <child link="${model_name}-hat" />
-            <axis rpy="0 0 0" xyz="0 0 1"/>
-        </joint>
-        <link name="${model_name}-hat">
-            <visual>
-                <origin rpy="0 0 0" xyz="0 0 0"/>
-                <geometry>
-                    <cylinder length="${L_HAT}" radius="${R_HAT}"/>
-                </geometry>
-                <material name="red"/>
-            </visual>
-            <collision>
-                <origin rpy="0 0 0" xyz="0 0 0"/>
-                <geometry>
-                    <cylinder length="${L_HAT}" radius="${R_HAT}"/>
-                </geometry>
-            </collision>
-            <inertial>
-                <mass value="${M_HAT}"/>
-                <origin rpy="0 0 0" xyz="0 0 0.04"/>
-                <inertia ixx="${1/12*M_HAT*(3*R_HAT*R_HAT+L_HAT*L_HAT)}" ixy="0" ixz="0" iyy="${1/12*M_HAT*(3*R_HAT*R_HAT+L_HAT*L_HAT)}" iyz="0" izz="${1/2*M_HAT*R_HAT*R_HAT}"/>
-            </inertial>
-        </link>
-        <gazebo reference="${model_name}-hat">
-            <material>Gazebo/Red</material>
-            <dampingFactor>0.02</dampingFactor>
-            <maxVel>0.1</maxVel>
-            <minDepth>0.01</minDepth>
-            <selfCollide>true</selfCollide>
-            <mu1>0.99</mu1>
-            <mu2>0.99</mu2>
+            <material>Gazebo/Wood</material>
         </gazebo>
     </xacro:macro>
